File: hardware/power_12v.kicad_sch (KiCad schematic)
At the start: 0 parts

Commit message: Kicad şema düzenlemesi yapıldı.
Parts:
- added C3, C4: 10uf, Capacitor_SMD:C_1206_3216Metric, symbol Device:C
- added R4, R5: R, symbol Device:R
- added U1: LM1084IS-3.3/NOPB, TS3B, symbol drip-irrigation-sys-cc:LM1084IS-3.3_NOPB
Connections:
- net PWR_12V: now also C4.1, R5.2, U1.2 (Vout)
- net PWR_12V_GND: now also C3.2, C4.2, R4.1
- net PWR_SOURCE_VCC: now also C3.1, U1.3 (Vin)
- new net: R4.2, R5.1, U1.1 (ADJ/GND)
Other:
- note added: "POWER TO 12V Regulator"
Changed lines of the file:
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@@
 (kicad_sch (version 20230121) (generator eeschema)
   (paper "A4")
+  (junction (at 99.06 53.34) (diameter 0) (color 0 0 0 0)
+  )
+  (junction (at 127 57.15) (diameter 0) (color 0 0 0 0)
+  )
+  (junction (at 120.65 39.37) (diameter 0) (color 0 0 0 0)
+  )
+  (junction (at 59.69 35.56) (diameter 0) (color 0 0 0 0)
+  )
+  (junction (at 59.69 53.34) (diameter 0) (color 0 0 0 0)
+  )
+  (junction (at 127 39.37) (diameter 0) (color 0 0 0 0)
+  )
+  (junction (at 44.45 53.34) (diameter 0) (color 0 0 0 0)
+  )
+  (wire (pts (xy 252.73 57.15) (xy 127 57.15))
+    (stroke (width 0) (type default))
+  )
+  (wire (pts (xy 250.19 31.75) (xy 262.89 31.75))
+    (stroke (width 0) (type default))
+  )
+  (wire (pts (xy 99.06 53.34) (xy 99.06 45.72))
+    (stroke (width 0) (type default))
+  )
+  (wire (pts (xy 59.69 35.56) (xy 59.69 45.72))
+    (stroke (width 0) (type default))
+  )
+  (wire (pts (xy 44.45 57.15) (xy 127 57.15))
+    (stroke (width 0) (type default))
+  )
+  (wire (pts (xy 36.83 35.56) (xy 59.69 35.56))
+    (stroke (width 0) (type default))
+  )
+  (wire (pts (xy 99.06 53.34) (xy 106.68 53.34))
+    (stroke (width 0) (type default))
+  )
+  (wire (pts (xy 114.3 53.34) (xy 120.65 53.34))
+    (stroke (width 0) (type default))
+  )
+  (wire (pts (xy 44.45 53.34) (xy 44.45 39.37))
+    (stroke (width 0) (type default))
+  )
+  (wire (pts (xy 59.69 53.34) (xy 73.66 53.34))
+    (stroke (width 0) (type default))
+  )
+  (wire (pts (xy 120.65 39.37) (xy 116.84 39.37))
+    (stroke (width 0) (type default))
+  )
+  (wire (pts (xy 68.58 35.56) (xy 68.58 36.83))
+    (stroke (width 0) (type default))
+  )
+  (wire (pts (xy 120.65 53.34) (xy 120.65 39.37))
+    (stroke (width 0) (type default))
+  )
+  (wire (pts (xy 252.73 34.29) (xy 252.73 57.15))
+    (stroke (width 0) (type default))
+  )
+  (wire (pts (xy 127 39.37) (xy 250.19 39.37))
+    (stroke (width 0) (type default))
+  )
+  (wire (pts (xy 44.45 53.34) (xy 44.45 57.15))
+    (stroke (width 0) (type default))
+  )
+  (wire (pts (xy 44.45 39.37) (xy 36.83 39.37))
+    (stroke (width 0) (type default))
+  )
+  (wire (pts (xy 99.06 45.72) (xy 124.46 45.72))
+    (stroke (width 0) (type default))
+  )
+  (wire (pts (xy 120.65 39.37) (xy 127 39.37))
+    (stroke (width 0) (type default))
+  )
+  (wire (pts (xy 124.46 45.72) (xy 124.46 36.83))
+    (stroke (width 0) (type default))
+  )
+  (wire (pts (xy 250.19 39.37) (xy 250.19 31.75))
+    (stroke (width 0) (type default))
+  )
+  (wire (pts (xy 81.28 53.34) (xy 99.06 53.34))
+    (stroke (width 0) (type default))
+  )
+  (wire (pts (xy 127 39.37) (xy 127 49.53))
+    (stroke (width 0) (type default))
+  )
+  (wire (pts (xy 124.46 36.83) (xy 116.84 36.83))
+    (stroke (width 0) (type default))
+  )
+  (wire (pts (xy 59.69 35.56) (xy 68.58 35.56))
+    (stroke (width 0) (type default))
+  )
+  (wire (pts (xy 59.69 53.34) (xy 44.45 53.34))
+    (stroke (width 0) (type default))
+  )
+  (wire (pts (xy 262.89 34.29) (xy 252.73 34.29))
+    (stroke (width 0) (type default))
+  )
+  (text "POWER TO 12V Regulator" (at 82.55 19.05 0)
+    (effects (font (size 1.27 1.27)) (justify left bottom))
+  )
   (hierarchical_label "PWR_SOURCE_VCC" (shape output) (at 36.83 35.56 180) (fields_autoplaced)
     (effects (font (size 1.27 1.27)) (justify right))
@@
     (effects (font (size 1.27 1.27)) (justify right))
   )
+  (symbol (lib_id "Device:R") (at 110.49 53.34 90) (unit 1)
+    (in_bom yes) (on_board yes) (dnp no) (fields_autoplaced)
+    (property "Reference" "R5" (at 110.49 46.99 90)
+      (effects (font (size 1.27 1.27)))
+    )
+    (property "Value" "R" (at 110.49 49.53 90)
+      (effects (font (size 1.27 1.27)))
+    )
+    (property "Footprint" "" (at 110.49 55.118 90)
+      (effects (font (size 1.27 1.27)) hide)
+    )
+    (property "Datasheet" "~" (at 110.49 53.34 0)
+      (effects (font (size 1.27 1.27)) hide)
+    )
+    (pin "1")
+    (pin "2")
+    (instances
+      (project "drip-irrigation-sys-cc"
+        (path "/41708c1e-19b2-4374-83f2-108076d82b45/4f778b49-8d1a-4c8f-a914-ecde21a56ebf/e37c023e-02fa-486d-a289-4e5112af51b8"
+          (reference "R5") (unit 1)
+        )
+      )
+    )
+  )
+  (symbol (lib_id "Device:C") (at 127 53.34 0) (unit 1)
+    (in_bom yes) (on_board yes) (dnp no) (fields_autoplaced)
+    (property "Reference" "C4" (at 130.81 52.07 0)
+      (effects (font (size 1.27 1.27)) (justify left))
+    )
+    (property "Value" "10uf" (at 130.81 54.61 0)
+      (effects (font (size 1.27 1.27)) (justify left))
+    )
+    (property "Footprint" "Capacitor_SMD:C_1206_3216Metric" (at 127.9652 57.15 0)
+      (effects (font (size 1.27 1.27)) hide)
+    )
+    (property "Datasheet" "~" (at 127 53.34 0)
+      (effects (font (size 1.27 1.27)) hide)
+    )
+    (property "Digikey" "478-3127-6-ND" (at 127 53.34 0)
+      (effects (font (size 1.27 1.27)) hide)
+    )
+    (pin "1")
+    (pin "2")
+    (instances
+      (project "drip-irrigation-sys-cc"
+        (path "/41708c1e-19b2-4374-83f2-108076d82b45/4f778b49-8d1a-4c8f-a914-ecde21a56ebf/e37c023e-02fa-486d-a289-4e5112af51b8"
+          (reference "C4") (unit 1)
+        )
+      )
+    )
+  )
+  (symbol (lib_id "drip-irrigation-sys-cc:LM1084IS-3.3_NOPB") (at 116.84 36.83 0) (mirror y) (unit 1)
+    (in_bom yes) (on_board yes) (dnp no)
+    (property "Reference" "U1" (at 92.71 26.67 0)
+      (effects (font (size 1.524 1.524)))
+    )
+    (property "Value" "LM1084IS-3.3/NOPB" (at 92.71 29.21 0)
+      (effects (font (size 1.524 1.524)))
+    )
+    (property "Footprint" "TS3B" (at 116.84 36.83 0)
+      (effects (font (size 1.27 1.27) italic) hide)
+    )
+    (property "Datasheet" "LM1084IS-3.3/NOPB" (at 116.84 36.83 0)
+      (effects (font (size 1.27 1.27) italic) hide)
+    )
+    (pin "1")
+    (pin "2")
+    (pin "3")
+    (pin "4")
+    (instances
+      (project "drip-irrigation-sys-cc"
+        (path "/41708c1e-19b2-4374-83f2-108076d82b45/4f778b49-8d1a-4c8f-a914-ecde21a56ebf/e37c023e-02fa-486d-a289-4e5112af51b8"
+          (reference "U1") (unit 1)
+        )
+      )
+    )
+  )
+  (symbol (lib_id "Device:R") (at 77.47 53.34 90) (unit 1)
+    (in_bom yes) (on_board yes) (dnp no) (fields_autoplaced)
+    (property "Reference" "R4" (at 77.47 46.99 90)
+      (effects (font (size 1.27 1.27)))
+    )
+    (property "Value" "R" (at 77.47 49.53 90)
+      (effects (font (size 1.27 1.27)))
+    )
+    (property "Footprint" "" (at 77.47 55.118 90)
+      (effects (font (size 1.27 1.27)) hide)
+    )
+    (property "Datasheet" "~" (at 77.47 53.34 0)
+      (effects (font (size 1.27 1.27)) hide)
+    )
+    (pin "1")
+    (pin "2")
+    (instances
+      (project "drip-irrigation-sys-cc"
+        (path "/41708c1e-19b2-4374-83f2-108076d82b45/4f778b49-8d1a-4c8f-a914-ecde21a56ebf/e37c023e-02fa-486d-a289-4e5112af51b8"
+          (reference "R4") (unit 1)
+        )
+      )
+    )
+  )
+  (symbol (lib_id "Device:C") (at 59.69 49.53 0) (unit 1)
+    (in_bom yes) (on_board yes) (dnp no) (fields_autoplaced)
+    (property "Reference" "C3" (at 63.5 48.26 0)
+      (effects (font (size 1.27 1.27)) (justify left))
+    )
+    (property "Value" "10uf" (at 63.5 50.8 0)
+      (effects (font (size 1.27 1.27)) (justify left))
+    )
+    (property "Footprint" "Capacitor_SMD:C_1206_3216Metric" (at 60.6552 53.34 0)
+      (effects (font (size 1.27 1.27)) hide)
+    )
+    (property "Datasheet" "~" (at 59.69 49.53 0)
+      (effects (font (size 1.27 1.27)) hide)
+    )
+    (property "Digikey" "478-3127-6-ND" (at 59.69 49.53 0)
+      (effects (font (size 1.27 1.27)) hide)
+    )
+    (pin "1")
+    (pin "2")
+    (instances
+      (project "drip-irrigation-sys-cc"
+        (path "/41708c1e-19b2-4374-83f2-108076d82b45/4f778b49-8d1a-4c8f-a914-ecde21a56ebf/e37c023e-02fa-486d-a289-4e5112af51b8"
+          (reference "C3") (unit 1)
+        )
+      )
+    )
+  )
 )

Commit message: Kicad şema düzenlemesi yapıldı.
Connections:
- net PWR_12V renamed +12V
- net PWR_12V_GND renamed GND
Changed lines of the file:
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@@
 (kicad_sch (version 20230121) (generator eeschema)
   (paper "A4")
+  (junction (at 127 57.15) (diameter 0) (color 0 0 0 0)
+  )
   (junction (at 99.06 53.34) (diameter 0) (color 0 0 0 0)
-  )
-  (junction (at 127 57.15) (diameter 0) (color 0 0 0 0)
   )
   (junction (at 120.65 39.37) (diameter 0) (color 0 0 0 0)
@@
   )
   (junction (at 44.45 53.34) (diameter 0) (color 0 0 0 0)
-  )
-  (wire (pts (xy 252.73 57.15) (xy 127 57.15))
-    (stroke (width 0) (type default))
-  )
-  (wire (pts (xy 250.19 31.75) (xy 262.89 31.75))
-    (stroke (width 0) (type default))
   )
   (wire (pts (xy 99.06 53.34) (xy 99.06 45.72))
@@
     (stroke (width 0) (type default))
   )
+  (wire (pts (xy 127 57.15) (xy 127 60.96))
+    (stroke (width 0) (type default))
+  )
   (wire (pts (xy 59.69 53.34) (xy 73.66 53.34))
     (stroke (width 0) (type default))
   )
   (wire (pts (xy 120.65 39.37) (xy 116.84 39.37))
+    (stroke (width 0) (type default))
+  )
+  (wire (pts (xy 127 39.37) (xy 152.4 39.37))
     (stroke (width 0) (type default))
   )
@@
     (stroke (width 0) (type default))
   )
-  (wire (pts (xy 252.73 34.29) (xy 252.73 57.15))
-    (stroke (width 0) (type default))
-  )
-  (wire (pts (xy 127 39.37) (xy 250.19 39.37))
+  (wire (pts (xy 152.4 33.02) (xy 152.4 39.37))
     (stroke (width 0) (type default))
   )
@@
     (stroke (width 0) (type default))
   )
-  (wire (pts (xy 250.19 39.37) (xy 250.19 31.75))
-    (stroke (width 0) (type default))
-  )
   (wire (pts (xy 81.28 53.34) (xy 99.06 53.34))
     (stroke (width 0) (type default))
@@
     (stroke (width 0) (type default))
   )
-  (wire (pts (xy 262.89 34.29) (xy 252.73 34.29))
-    (stroke (width 0) (type default))
-  )
   (text "POWER TO 12V Regulator" (at 82.55 19.05 0)
     (effects (font (size 1.27 1.27)) (justify left bottom))
@@
     (effects (font (size 1.27 1.27)) (justify right))
   )
-  (hierarchical_label "PWR_12V" (shape output) (at 262.89 31.75 0) (fields_autoplaced)
-    (effects (font (size 1.27 1.27)) (justify left))
-  )
-  (hierarchical_label "PWR_12V_GND" (shape output) (at 262.89 34.29 0) (fields_autoplaced)
-    (effects (font (size 1.27 1.27)) (justify left))
-  )
   (hierarchical_label "PWR_SOURCE_GND" (shape input) (at 36.83 39.37 180) (fields_autoplaced)
     (effects (font (size 1.27 1.27)) (justify right))
+  )
+  (symbol (lib_id "power:+12V") (at 152.4 33.02 0) (unit 1)
+    (in_bom yes) (on_board yes) (dnp no) (fields_autoplaced)
+    (property "Reference" "#PWR011" (at 152.4 36.83 0)
+      (effects (font (size 1.27 1.27)) hide)
+    )
+    (property "Value" "+12V" (at 152.4 27.94 0)
+      (effects (font (size 1.27 1.27)))
+    )
+    (property "Footprint" "" (at 152.4 33.02 0)
+      (effects (font (size 1.27 1.27)) hide)
+    )
+    (property "Datasheet" "" (at 152.4 33.02 0)
+      (effects (font (size 1.27 1.27)) hide)
+    )
+    (pin "1")
+    (instances
+      (project "drip-irrigation-sys-cc"
+        (path "/41708c1e-19b2-4374-83f2-108076d82b45"
+          (reference "#PWR011") (unit 1)
+        )
+        (path "/41708c1e-19b2-4374-83f2-108076d82b45/4f778b49-8d1a-4c8f-a914-ecde21a56ebf"
+          (reference "#PWR011") (unit 1)
+        )
+        (path "/41708c1e-19b2-4374-83f2-108076d82b45/4f778b49-8d1a-4c8f-a914-ecde21a56ebf/e37c023e-02fa-486d-a289-4e5112af51b8"
+          (reference "#PWR011") (unit 1)
+        )
+      )
+    )
   )
   (symbol (lib_id "Device:R") (at 110.49 53.34 90) (unit 1)
@@
         )
       )
+    )
+  )
+  (symbol (lib_id "power:GND") (at 127 60.96 0) (unit 1)
+    (in_bom yes) (on_board yes) (dnp no) (fields_autoplaced)
+    (property "Reference" "#PWR013" (at 127 67.31 0)
+      (effects (font (size 1.27 1.27)) hide)
+    )
+    (property "Value" "GND" (at 127 66.04 0)
+      (effects (font (size 1.27 1.27)))
+    )
+    (property "Footprint" "" (at 127 60.96 0)
+      (effects (font (size 1.27 1.27)) hide)
+    )
+    (property "Datasheet" "" (at 127 60.96 0)
+      (effects (font (size 1.27 1.27)) hide)
+    )
+    (pin "1")
+    (instances
+      (project "drip-irrigation-sys-cc"
+        (path "/41708c1e-19b2-4374-83f2-108076d82b45"
+          (reference "#PWR013") (unit 1)
+        )
+        (path "/41708c1e-19b2-4374-83f2-108076d82b45/4f778b49-8d1a-4c8f-a914-ecde21a56ebf"
+          (reference "#PWR013") (unit 1)
+        )
+        (path "/41708c1e-19b2-4374-83f2-108076d82b45/4f778b49-8d1a-4c8f-a914-ecde21a56ebf/e37c023e-02fa-486d-a289-4e5112af51b8"
+          (reference "#PWR014") (unit 1)
+        )
+      )
