File: hardware/adc.kicad_sch (KiCad schematic)
At the start: 0 parts

Commit message: Kicad şema düzenlemesi yapıldı.
Parts:
- added C13: 100nf, symbol Device:C
Connections:
- new net MCU_ADC: C13.2
- new net PRESSURE_SENSOR_ANALOG_SIGNAL: C13.1
Changed lines of the file:
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@@
 (kicad_sch (version 20230121) (generator eeschema)
   (paper "A4")
+  (wire (pts (xy 52.07 30.48) (xy 85.09 30.48))
+    (stroke (width 0) (type default))
+  )
+  (wire (pts (xy 92.71 30.48) (xy 121.92 30.48))
+    (stroke (width 0) (type default))
+  )
+  (hierarchical_label "PRESSURE_SENSOR_ANALOG_SIGNAL" (shape input) (at 52.07 30.48 180) (fields_autoplaced)
+    (effects (font (size 1.27 1.27)) (justify right))
+  )
+  (hierarchical_label "MCU_ADC" (shape output) (at 121.92 30.48 0) (fields_autoplaced)
+    (effects (font (size 1.27 1.27)) (justify left))
+  )
+  (symbol (lib_id "Device:C") (at 88.9 30.48 90) (unit 1)
+    (in_bom yes) (on_board yes) (dnp no) (fields_autoplaced)
+    (property "Reference" "C13" (at 88.9 22.86 90)
+      (effects (font (size 1.27 1.27)))
+    )
+    (property "Value" "100nf" (at 88.9 25.4 90)
+      (effects (font (size 1.27 1.27)))
+    )
+    (property "Footprint" "" (at 92.71 29.5148 0)
+      (effects (font (size 1.27 1.27)) hide)
+    )
+    (property "Datasheet" "~" (at 88.9 30.48 0)
+      (effects (font (size 1.27 1.27)) hide)
+    )
+    (pin "1")
+    (pin "2")
+    (instances
+      (project "drip-irrigation-sys-cc"
+        (path "/41708c1e-19b2-4374-83f2-108076d82b45/8c94c97b-f919-45ea-a17c-2e0bf75da6f4"
+          (reference "C13") (unit 1)
+        )
+      )
+    )
+  )
 )

Commit message: Kicad şema düzenlemesi yapıldı.
Parts:
- removed C13: 100nf, symbol Device:C
- added R8: 1K, Resistor_SMD:R_0603_1608Metric, symbol Device:R
- added R9: 2.74K, Resistor_SMD:R_0603_1608Metric, symbol Device:R
Connections:
- net MCU_ADC: now also R8.2, R9.1
- net PRESSURE_SENSOR_ANALOG_SIGNAL: now also R8.1
- new net GND: R9.2
Changed lines of the file:
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@@
 (kicad_sch (version 20230121) (generator eeschema)
   (paper "A4")
-  (wire (pts (xy 52.07 30.48) (xy 85.09 30.48))
+  (junction (at 78.74 58.42) (diameter 0) (color 0 0 0 0)
+  )
+  (wire (pts (xy 92.71 58.42) (xy 101.6 58.42))
     (stroke (width 0) (type default))
   )
-  (wire (pts (xy 92.71 30.48) (xy 121.92 30.48))
+  (wire (pts (xy 78.74 43.18) (xy 78.74 58.42))
     (stroke (width 0) (type default))
   )
-  (hierarchical_label "PRESSURE_SENSOR_ANALOG_SIGNAL" (shape input) (at 52.07 30.48 180) (fields_autoplaced)
+  (wire (pts (xy 52.07 58.42) (xy 64.77 58.42))
+    (stroke (width 0) (type default))
+  )
+  (wire (pts (xy 72.39 58.42) (xy 78.74 58.42))
+    (stroke (width 0) (type default))
+  )
+  (wire (pts (xy 78.74 58.42) (xy 85.09 58.42))
+    (stroke (width 0) (type default))
+  )
+  (wire (pts (xy 101.6 58.42) (xy 101.6 63.5))
+    (stroke (width 0) (type default))
+  )
+  (hierarchical_label "PRESSURE_SENSOR_ANALOG_SIGNAL" (shape input) (at 52.07 58.42 180) (fields_autoplaced)
     (effects (font (size 1.27 1.27)) (justify right))
   )
-  (hierarchical_label "MCU_ADC" (shape output) (at 121.92 30.48 0) (fields_autoplaced)
+  (hierarchical_label "MCU_ADC" (shape output) (at 78.74 43.18 90) (fields_autoplaced)
     (effects (font (size 1.27 1.27)) (justify left))
   )
-  (symbol (lib_id "Device:C") (at 88.9 30.48 90) (unit 1)
+  (symbol (lib_id "Device:R") (at 68.58 58.42 90) (unit 1)
     (in_bom yes) (on_board yes) (dnp no) (fields_autoplaced)
-    (property "Reference" "C13" (at 88.9 22.86 90)
+    (property "Reference" "R8" (at 68.58 52.07 90)
       (effects (font (size 1.27 1.27)))
     )
-    (property "Value" "100nf" (at 88.9 25.4 90)
+    (property "Value" "1K" (at 68.58 54.61 90)
       (effects (font (size 1.27 1.27)))
     )
-    (property "Footprint" "" (at 92.71 29.5148 0)
+    (property "Footprint" "Resistor_SMD:R_0603_1608Metric" (at 68.58 60.198 90)
       (effects (font (size 1.27 1.27)) hide)
     )
-    (property "Datasheet" "~" (at 88.9 30.48 0)
+    (property "Datasheet" "~" (at 68.58 58.42 0)
+      (effects (font (size 1.27 1.27)) hide)
+    )
+    (property "Digikey" "311-1.00KHRDKR-ND" (at 68.58 58.42 90)
       (effects (font (size 1.27 1.27)) hide)
     )
@@
       (project "drip-irrigation-sys-cc"
         (path "/41708c1e-19b2-4374-83f2-108076d82b45/8c94c97b-f919-45ea-a17c-2e0bf75da6f4"
-          (reference "C13") (unit 1)
+          (reference "R8") (unit 1)
         )
       )
+    )
+  )
+  (symbol (lib_id "Device:R") (at 88.9 58.42 90) (unit 1)
+    (in_bom yes) (on_board yes) (dnp no) (fields_autoplaced)
+    (property "Reference" "R9" (at 88.9 52.07 90)
+      (effects (font (size 1.27 1.27)))
+    )
+    (property "Value" "2.74K" (at 88.9 54.61 90)
+      (effects (font (size 1.27 1.27)))
+    )
+    (property "Footprint" "Resistor_SMD:R_0603_1608Metric" (at 88.9 60.198 90)
+      (effects (font (size 1.27 1.27)) hide)
+    )
+    (property "Datasheet" "~" (at 88.9 58.42 0)
+      (effects (font (size 1.27 1.27)) hide)
+    )
+    (property "Digikey" "311-2.74KHRDKR-ND" (at 88.9 58.42 90)
+      (effects (font (size 1.27 1.27)) hide)
+    )
+    (pin "1")
+    (pin "2")
+    (instances
+      (project "drip-irrigation-sys-cc"
+        (path "/41708c1e-19b2-4374-83f2-108076d82b45/8c94c97b-f919-45ea-a17c-2e0bf75da6f4"
+          (reference "R9") (unit 1)
+        )
+      )
+    )
+  )
+  (symbol (lib_id "power:GND") (at 101.6 63.5 0) (unit 1)
+    (in_bom yes) (on_board yes) (dnp no) (fields_autoplaced)
+    (property "Reference" "#PWR018" (at 101.6 69.85 0)
+      (effects (font (size 1.27 1.27)) hide)
+    )
+    (property "Value" "GND" (at 101.6 68.58 0)
+      (effects (font (size 1.27 1.27)))
+    )
+    (property "Footprint" "" (at 101.6 63.5 0)
+      (effects (font (size 1.27 1.27)) hide)
+    )
+    (property "Datasheet" "" (at 101.6 63.5 0)
+      (effects (font (size 1.27 1.27)) hide)
+    )
+    (pin "1")
+    (instances
+      (project "drip-irrigation-sys-cc"
+        (path "/41708c1e-19b2-4374-83f2-108076d82b45/8c94c97b-f919-45ea-a17c-2e0bf75da6f4"
+          (reference "#PWR018") (unit 1)
+        )
+      )

Commit message: Kicad şema düzenlemesi yapıldı.
Parts:
- renumbered R8 to R12, R9 to R13
Changed lines of the file:
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@@
   (symbol (lib_id "Device:R") (at 68.58 58.42 90) (unit 1)
     (in_bom yes) (on_board yes) (dnp no) (fields_autoplaced)
-    (property "Reference" "R8" (at 68.58 52.07 90)
+    (property "Reference" "R12" (at 68.58 52.07 90)
       (effects (font (size 1.27 1.27)))
     )
@@
       (project "drip-irrigation-sys-cc"
         (path "/41708c1e-19b2-4374-83f2-108076d82b45/8c94c97b-f919-45ea-a17c-2e0bf75da6f4"
-          (reference "R8") (unit 1)
+          (reference "R12") (unit 1)
         )
       )
@@
   (symbol (lib_id "Device:R") (at 88.9 58.42 90) (unit 1)
     (in_bom yes) (on_board yes) (dnp no) (fields_autoplaced)
-    (property "Reference" "R9" (at 88.9 52.07 90)
+    (property "Reference" "R13" (at 88.9 52.07 90)
       (effects (font (size 1.27 1.27)))
     )
@@
       (project "drip-irrigation-sys-cc"
         (path "/41708c1e-19b2-4374-83f2-108076d82b45/8c94c97b-f919-45ea-a17c-2e0bf75da6f4"
-          (reference "R9") (unit 1)
+          (reference "R13") (unit 1)
         )
       )
@@
   (symbol (lib_id "power:GND") (at 101.6 63.5 0) (unit 1)
     (in_bom yes) (on_board yes) (dnp no) (fields_autoplaced)
-    (property "Reference" "#PWR018" (at 101.6 69.85 0)
+    (property "Reference" "#PWR031" (at 101.6 69.85 0)
       (effects (font (size 1.27 1.27)) hide)
     )
@@
       (project "drip-irrigation-sys-cc"
         (path "/41708c1e-19b2-4374-83f2-108076d82b45/8c94c97b-f919-45ea-a17c-2e0bf75da6f4"
-          (reference "#PWR018") (unit 1)
+          (reference "#PWR031") (unit 1)
         )
       )
