File: hardware/drip-irrigation-sys-cc.kicad_sch (KiCad schematic)
At the start: 29 parts, among them J1 RELAY, J2 PWR, J3 PRESSURE_SENSOR, J4 USB_A, J8 UJ2-AV-4-SMT-TR, J9 Conn_02x01, SW1 BTN_DEACTIVE, SW2 BTN_IO, SW3 BTN_ACTIVE

Commit message: Kicad şema düzenlemesi yapıldı.
Parts:
- removed J8: UJ2-AV-4-SMT-TR, CONN4X1_UJ2-AV-4-SMT-TR_CUD, symbol drip-irrigation-sys-cc:UJ2-AV-4-SMT-TR
- C1: renamed from C19; footprint Capacitor_SMD:C_1206_3216Metric -> Capacitor_SMD:C_0805_2012Metric; Digikey 5440-FN31X103K500PXGTR-ND -> (none)
- C?: renamed from C8; footprint Capacitor_SMD:C_0201_0603Metric -> Capacitor_SMD:C_0805_2012Metric; Digikey 490-3167-2-ND -> (none)
- C?: renamed from C7; footprint Capacitor_SMD:C_0201_0603Metric -> Capacitor_SMD:C_0805_2012Metric; Digikey 490-3167-2-ND -> (none)
- C?: renamed from C9; footprint Capacitor_SMD:C_0201_0603Metric -> Capacitor_SMD:C_0805_2012Metric; Digikey 490-3167-2-ND -> (none)
- D1: renamed from D9; footprint LED_SMD:LED_0603_1608Metric -> LED_SMD:LED_0805_2012Metric; Digikey 67-SML-LXFT0603GC-TR-ND -> (none)
- D2: renamed from D8; footprint LED_SMD:LED_0603_1608Metric -> LED_SMD:LED_0805_2012Metric; Digikey 67-SML-LXFT0603GC-TR-ND -> (none)
- D3: renamed from D7; footprint LED_SMD:LED_1206_3216Metric -> LED_SMD:LED_0805_2012Metric; Digikey 754-AP3216IDTR-ND -> (none)
- J4: renamed from J9; footprint Connector_PinHeader_1.00mm:PinHeader_1x02_P1.00mm_Vertical -> Connector_Phoenix_MC:PhoenixContact_MCV_1,5_2-G-3.81_1x02_P3.81mm_Vertical
- R1: renamed from R14; footprint Resistor_SMD:R_0402_1005Metric -> Resistor_SMD:R_0603_1608Metric; Digikey 2577-AS02FTE3300TR-ND -> (none)
- R2: renamed from R15; footprint Resistor_SMD:R_0402_1005Metric -> Resistor_SMD:R_0603_1608Metric; Digikey 2577-AS02FTE3300TR-ND -> (none)
- R3: renamed from R16; footprint Resistor_SMD:R_0402_1005Metric -> Resistor_SMD:R_0603_1608Metric; Digikey 2577-AS02FTE3300TR-ND -> (none)
- R4: renamed from R1; footprint Resistor_SMD:R_0402_1005Metric -> Resistor_SMD:R_0603_1608Metric; Digikey 1276-3431-2-ND -> (none)
- R6: renamed from R3; footprint Resistor_SMD:R_0402_1005Metric -> Resistor_SMD:R_0603_1608Metric; Digikey 1276-3431-2-ND -> (none)
- R8: renamed from R5; footprint Resistor_SMD:R_0402_1005Metric -> Resistor_SMD:R_0603_1608Metric; Digikey 1276-3431-2-ND -> (none)
- renumbered J2 to J1, J4 to J2, J1 to J5, R2 to R5, R4 to R7, R6 to R9
Other:
- sheet GSM_Module ports: added 5V_Input, UART_RX, UART_TX; removed 5V_INPUT, uart1_rx, uart1_tx
- sheet RS-485 ports: added USART2_RX, USART2_TX; removed RS485_A, RS485_B
