File: hardware/drip-irrigation-sys-cc.kicad_sch (KiCad schematic)
At the start: 28 parts, among them J1 PWR, J2 USB_A, J3 PRESSURE_SENSOR, J4 Conn_02x01, J5 RELAY, SW1 BTN_DEACTIVE, SW2 BTN_IO, SW3 BTN_ACTIVE

Commit message: PCB düzenleme.
Parts:
- C1: Digikey (none) -> 0805B103K251DC
- C? (x3): Digikey (none) -> 3372-0805B104K500BDTR-ND
- D1, D2: Digikey (none) -> 3372-0805YGBD008S01TR-ND
- D3: Digikey (none) -> 3372-0805RBD0070S01TR-ND
- R1, R2, R3: Digikey (none) -> A121525DKR-ND
Changed lines of the file:
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@@
       (effects (font (size 1.27 1.27)) hide)
     )
-    (property "Digikey" "" (at 245.11 143.51 0)
+    (property "Digikey" "3372-0805B104K500BDTR-ND" (at 245.11 143.51 0)
       (effects (font (size 1.27 1.27)) hide)
     )
@@
       (effects (font (size 1.27 1.27)) hide)
     )
-    (property "Digikey" "" (at 66.04 69.85 0)
+    (property "Digikey" "A121525DKR-ND" (at 66.04 69.85 0)
       (effects (font (size 1.27 1.27)) hide)
     )
@@
       (effects (font (size 1.27 1.27)) hide)
     )
-    (property "Digikey" "" (at 113.03 63.5 0)
+    (property "Digikey" "A121525DKR-ND" (at 113.03 63.5 0)
       (effects (font (size 1.27 1.27)) hide)
     )
@@
       (effects (font (size 1.27 1.27)) hide)
     )
-    (property "Digikey" "" (at 125.73 63.5 0)
+    (property "Digikey" "3372-0805YGBD008S01TR-ND" (at 125.73 63.5 0)
       (effects (font (size 1.27 1.27)) hide)
     )
@@
       (effects (font (size 1.27 1.27)) hide)
     )
-    (property "Digikey" "" (at 171.45 66.04 0)
+    (property "Digikey" "A121525DKR-ND" (at 171.45 66.04 0)
       (effects (font (size 1.27 1.27)) hide)
     )
@@
       (effects (font (size 1.27 1.27)) hide)
     )
-    (property "Digikey" "" (at 38.1 154.94 0)
+    (property "Digikey" "0805B103K251DC" (at 38.1 154.94 0)
       (effects (font (size 1.27 1.27)) hide)
     )
@@
       (effects (font (size 1.27 1.27)) hide)
     )
-    (property "Digikey" "" (at 185.42 66.04 0)
+    (property "Digikey" "3372-0805RBD0070S01TR-ND" (at 185.42 66.04 0)
       (effects (font (size 1.27 1.27)) hide)
     )
@@
       (effects (font (size 1.27 1.27)) hide)
     )
-    (property "Digikey" "" (at 213.36 143.51 0)
+    (property "Digikey" "3372-0805B104K500BDTR-ND" (at 213.36 143.51 0)
       (effects (font (size 1.27 1.27)) hide)
     )
@@
       (effects (font (size 1.27 1.27)) hide)
     )
-    (property "Digikey" "" (at 266.7 143.51 0)
+    (property "Digikey" "3372-0805B104K500BDTR-ND" (at 266.7 143.51 0)
       (effects (font (size 1.27 1.27)) hide)
     )
@@
       (effects (font (size 1.27 1.27)) hide)
     )
-    (property "Digikey" "" (at 80.01 69.85 0)
-      (effects (font (size 1.27 1.27)) hide)
-    )
+    (property "Digikey" "3372-0805YGBD008S01TR-ND" (at 80.01 69.85 0)
+      (effects (font (size 1.27 1.27)) hide)
+    )
