File: hardware/exp.kicad_sch (KiCad schematic)
At the start: 1 part, among them J7 Conn_02x06_Top_Bottom

Commit message: Kicad şema düzenlemesi yapıldı.
Parts:
- renumbered J7 to J9
Connections:
- net +3.3V: now also J9.4 (Pin_4), J9.5 (Pin_5); no longer J9.12 (Pin_12)
- net GND: now also J9.12 (Pin_12); no longer J9.4 (Pin_4), J9.5 (Pin_5)
Changed lines of the file:
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@@
     (effects (font (size 1.27 1.27)) (justify left))
-  )
-  (symbol (lib_id "power:GND") (at 85.09 76.2 270) (unit 1)
-    (in_bom yes) (on_board yes) (dnp no) (fields_autoplaced)
-    (property "Reference" "#PWR064" (at 78.74 76.2 0)
-      (effects (font (size 1.27 1.27)) hide)
-    )
-    (property "Value" "GND" (at 81.28 76.2 90)
-      (effects (font (size 1.27 1.27)) (justify right))
-    )
-    (property "Footprint" "" (at 85.09 76.2 0)
-      (effects (font (size 1.27 1.27)) hide)
-    )
-    (property "Datasheet" "" (at 85.09 76.2 0)
-      (effects (font (size 1.27 1.27)) hide)
-    )
-    (pin "1")
-    (instances
-      (project "drip-irrigation-sys-cc"
-        (path "/41708c1e-19b2-4374-83f2-108076d82b45/615c9dda-6fc9-4083-94d9-1e6f9ee22c73"
-          (reference "#PWR064") (unit 1)
-        )
-      )
-    )
   )
   (symbol (lib_id "power:GND") (at 115.57 76.2 90) (mirror x) (unit 1)
     (in_bom yes) (on_board yes) (dnp no)
-    (property "Reference" "#PWR066" (at 121.92 76.2 0)
+    (property "Reference" "#PWR056" (at 121.92 76.2 0)
       (effects (font (size 1.27 1.27)) hide)
     )
@@
       (project "drip-irrigation-sys-cc"
         (path "/41708c1e-19b2-4374-83f2-108076d82b45/615c9dda-6fc9-4083-94d9-1e6f9ee22c73"
-          (reference "#PWR066") (unit 1)
+          (reference "#PWR056") (unit 1)
         )
       )
     )
   )
-  (symbol (lib_id "power:GND") (at 85.09 73.66 270) (unit 1)
-    (in_bom yes) (on_board yes) (dnp no) (fields_autoplaced)
-    (property "Reference" "#PWR065" (at 78.74 73.66 0)
+  (symbol (lib_id "power:GND") (at 115.57 78.74 90) (mirror x) (unit 1)
+    (in_bom yes) (on_board yes) (dnp no)
+    (property "Reference" "#PWR057" (at 121.92 78.74 0)
       (effects (font (size 1.27 1.27)) hide)
     )
-    (property "Value" "GND" (at 81.28 73.66 90)
+    (property "Value" "GND" (at 119.38 78.74 90)
       (effects (font (size 1.27 1.27)) (justify right))
     )
-    (property "Footprint" "" (at 85.09 73.66 0)
+    (property "Footprint" "" (at 115.57 78.74 0)
       (effects (font (size 1.27 1.27)) hide)
     )
-    (property "Datasheet" "" (at 85.09 73.66 0)
+    (property "Datasheet" "" (at 115.57 78.74 0)
       (effects (font (size 1.27 1.27)) hide)
     )
@@
       (project "drip-irrigation-sys-cc"
         (path "/41708c1e-19b2-4374-83f2-108076d82b45/615c9dda-6fc9-4083-94d9-1e6f9ee22c73"
-          (reference "#PWR065") (unit 1)
+          (reference "#PWR057") (unit 1)
         )
       )
@@
   (symbol (lib_id "Connector_Generic:Conn_02x06_Top_Bottom") (at 99.06 71.12 0) (unit 1)
     (in_bom yes) (on_board yes) (dnp no) (fields_autoplaced)
-    (property "Reference" "J7" (at 100.33 59.69 0)
+    (property "Reference" "J9" (at 100.33 59.69 0)
       (effects (font (size 1.27 1.27)))
     )
@@
       (project "drip-irrigation-sys-cc"
         (path "/41708c1e-19b2-4374-83f2-108076d82b45/615c9dda-6fc9-4083-94d9-1e6f9ee22c73"
-          (reference "J7") (unit 1)
+          (reference "J9") (unit 1)
         )
       )
     )
   )
-  (symbol (lib_id "power:+3.3V") (at 115.57 78.74 270) (unit 1)
-    (in_bom yes) (on_board yes) (dnp no) (fields_autoplaced)
-    (property "Reference" "#PWR063" (at 111.76 78.74 0)
+  (symbol (lib_id "power:+3.3V") (at 85.09 73.66 90) (mirror x) (unit 1)
+    (in_bom yes) (on_board yes) (dnp no)
+    (property "Reference" "#PWR053" (at 88.9 73.66 0)
       (effects (font (size 1.27 1.27)) hide)
     )
-    (property "Value" "+3.3V" (at 119.38 78.74 90)
+    (property "Value" "+3.3V" (at 81.28 73.66 90)
       (effects (font (size 1.27 1.27)) (justify left))
     )
-    (property "Footprint" "" (at 115.57 78.74 0)
+    (property "Footprint" "" (at 85.09 73.66 0)
       (effects (font (size 1.27 1.27)) hide)
     )
-    (property "Datasheet" "" (at 115.57 78.74 0)
+    (property "Datasheet" "" (at 85.09 73.66 0)
       (effects (font (size 1.27 1.27)) hide)
     )
@@
       (project "drip-irrigation-sys-cc"
         (path "/41708c1e-19b2-4374-83f2-108076d82b45/615c9dda-6fc9-4083-94d9-1e6f9ee22c73"
-          (reference "#PWR063") (unit 1)
+          (reference "#PWR053") (unit 1)
+        )
+      )
+    )
+  )
+  (symbol (lib_id "power:+3.3V") (at 85.09 76.2 90) (mirror x) (unit 1)
+    (in_bom yes) (on_board yes) (dnp no)
+    (property "Reference" "#PWR054" (at 88.9 76.2 0)
+      (effects (font (size 1.27 1.27)) hide)
+    )
+    (property "Value" "+3.3V" (at 81.28 76.2 90)
+      (effects (font (size 1.27 1.27)) (justify left))
+    )
+    (property "Footprint" "" (at 85.09 76.2 0)
+      (effects (font (size 1.27 1.27)) hide)
+    )
+    (property "Datasheet" "" (at 85.09 76.2 0)
+      (effects (font (size 1.27 1.27)) hide)
+    )
+    (pin "1")
+    (instances
+      (project "drip-irrigation-sys-cc"
+        (path "/41708c1e-19b2-4374-83f2-108076d82b45/615c9dda-6fc9-4083-94d9-1e6f9ee22c73"
+          (reference "#PWR054") (unit 1)
         )
       )
@@
   (symbol (lib_id "power:+5V") (at 85.09 78.74 90) (unit 1)
     (in_bom yes) (on_board yes) (dnp no) (fields_autoplaced)
-    (property "Reference" "#PWR062" (at 88.9 78.74 0)
+    (property "Reference" "#PWR055" (at 88.9 78.74 0)
       (effects (font (size 1.27 1.27)) hide)
     )
@@
       (project "drip-irrigation-sys-cc"
         (path "/41708c1e-19b2-4374-83f2-108076d82b45/615c9dda-6fc9-4083-94d9-1e6f9ee22c73"
-          (reference "#PWR062") (unit 1)
+          (reference "#PWR055") (unit 1)
         )
       )
