File: hardware/power_5v.kicad_sch (KiCad schematic)
At the start: 5 parts, among them U5 LM2576-5.0WU-TR

Commit message: Kicad şema düzenlemesi.
Parts:
- L2: footprint drip-irrigation-sys-cc:IND_HCTI-220-5.8 -> Inductor_SMD:L_12x12mm_H8mm; Digikey 595-1734-ND -> 553-3620-6-ND
Changed lines of the file:
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@@
       (effects (font (size 1.27 1.27)))
     )
-    (property "Footprint" "drip-irrigation-sys-cc:IND_HCTI-220-5.8" (at 226.06 50.8 0)
+    (property "Footprint" "Inductor_SMD:L_12x12mm_H8mm" (at 226.06 50.8 0)
       (effects (font (size 1.27 1.27)) hide)
     )
@@
       (effects (font (size 1.27 1.27)) hide)
     )
-    (property "Digikey" "595-1734-ND" (at 226.06 50.8 90)
+    (property "Digikey" "553-3620-6-ND" (at 226.06 50.8 90)
       (effects (font (size 1.27 1.27)) hide)
     )
