File: hardware/relay.kicad_sch (KiCad schematic)
At the start: 4 parts, among them K1 Relay_SPDT, Q3 NPN

Commit message: Kicad şema düzenlemesi yapıldı.
Parts:
- removed Q3: NPN, symbol Simulation_SPICE:NPN
- added Q1: MMBT3904-TP, SOT-23_MCC, symbol drip-irrigation-sys-cc:MMBT3904-TP
- K1: Digikey (none) -> Z3672-ND
- R7: value R -> 1K; footprint (none) -> Resistor_SMD:R_0603_1608Metric
Connections:
- net +5V: now also Q1.3
- net at C14.2: now also Q1.1
- net at K1.A1: now also Q1.2
Changed lines of the file:
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@@
-    )
-  )
-  (symbol (lib_id "Simulation_SPICE:NPN") (at 143.51 62.23 0) (unit 1)
-    (in_bom yes) (on_board yes) (dnp no) (fields_autoplaced)
-    (property "Reference" "Q3" (at 148.59 60.96 0)
-      (effects (font (size 1.27 1.27)) (justify left))
-    )
-    (property "Value" "NPN" (at 148.59 63.5 0)
-      (effects (font (size 1.27 1.27)) (justify left))
-    )
-    (property "Footprint" "" (at 207.01 62.23 0)
-      (effects (font (size 1.27 1.27)) hide)
-    )
-    (property "Datasheet" "~" (at 207.01 62.23 0)
-      (effects (font (size 1.27 1.27)) hide)
-    )
-    (property "Sim.Device" "NPN" (at 143.51 62.23 0)
-      (effects (font (size 1.27 1.27)) hide)
-    )
-    (property "Sim.Type" "GUMMELPOON" (at 143.51 62.23 0)
-      (effects (font (size 1.27 1.27)) hide)
-    )
-    (property "Sim.Pins" "1=C 2=B 3=E" (at 143.51 62.23 0)
-      (effects (font (size 1.27 1.27)) hide)
-    )
-    (pin "1")
-    (pin "2")
-    (pin "3")
-    (instances
-      (project "drip-irrigation-sys-cc"
-        (path "/41708c1e-19b2-4374-83f2-108076d82b45/202a1cab-a33b-4ef0-945c-8042c7ebf8be"
-          (reference "Q3") (unit 1)
-        )
-      )
     )
   )
@@
       (effects (font (size 1.27 1.27)))
     )
-    (property "Value" "R" (at 116.84 58.42 90)
+    (property "Value" "1K" (at 116.84 58.42 90)
       (effects (font (size 1.27 1.27)))
     )
-    (property "Footprint" "" (at 116.84 64.008 90)
+    (property "Footprint" "Resistor_SMD:R_0603_1608Metric" (at 116.84 64.008 90)
       (effects (font (size 1.27 1.27)) hide)
     )
@@
     )
   )
+  (symbol (lib_id "drip-irrigation-sys-cc:MMBT3904-TP") (at 138.43 62.23 0) (unit 1)
+    (in_bom yes) (on_board yes) (dnp no) (fields_autoplaced)
+    (property "Reference" "Q1" (at 148.59 60.96 0)
+      (effects (font (size 1.524 1.524)) (justify left))
+    )
+    (property "Value" "MMBT3904-TP" (at 148.59 63.5 0)
+      (effects (font (size 1.524 1.524)) (justify left))
+    )
+    (property "Footprint" "SOT-23_MCC" (at 138.43 62.23 0)
+      (effects (font (size 1.27 1.27) italic) hide)
+    )
+    (property "Datasheet" "MMBT3904-TP" (at 138.43 62.23 0)
+      (effects (font (size 1.27 1.27) italic) hide)
+    )
+    (pin "1")
+    (pin "2")
+    (pin "3")
+    (instances
+      (project "drip-irrigation-sys-cc"
+        (path "/41708c1e-19b2-4374-83f2-108076d82b45/202a1cab-a33b-4ef0-945c-8042c7ebf8be"
+          (reference "Q1") (unit 1)
+        )
+      )
+    )
+  )
   (symbol (lib_id "Relay:Relay_SPDT") (at 152.4 92.71 0) (unit 1)
     (in_bom yes) (on_board yes) (dnp no) (fields_autoplaced)
@@
       (effects (font (size 1.27 1.27)) hide)
     )
+    (property "Digikey" "Z3672-ND" (at 152.4 92.71 0)
+      (effects (font (size 1.27 1.27)) hide)
+    )

Commit message: Kicad şema düzenlemesi yapıldı.
Parts:
- C21: renamed from C14; footprint Capacitor_SMD:C_0201_0603Metric -> Capacitor_SMD:C_0805_2012Metric; Digikey 490-3167-2-ND -> (none)
- Q1: Digikey (none) -> MMBT3904TPMSTR-ND
- renumbered R7 to R17
Changed lines of the file:
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@@
   (symbol (lib_id "power:+5V") (at 146.05 24.13 0) (unit 1)
     (in_bom yes) (on_board yes) (dnp no) (fields_autoplaced)
-    (property "Reference" "#PWR013" (at 146.05 27.94 0)
+    (property "Reference" "#PWR040" (at 146.05 27.94 0)
       (effects (font (size 1.27 1.27)) hide)
     )
@@
       (project "drip-irrigation-sys-cc"
         (path "/41708c1e-19b2-4374-83f2-108076d82b45/202a1cab-a33b-4ef0-945c-8042c7ebf8be"
-          (reference "#PWR013") (unit 1)
+          (reference "#PWR040") (unit 1)
         )
       )
@@
   (symbol (lib_id "power:GND") (at 147.32 101.6 0) (unit 1)
     (in_bom yes) (on_board yes) (dnp no) (fields_autoplaced)
-    (property "Reference" "#PWR012" (at 147.32 107.95 0)
+    (property "Reference" "#PWR041" (at 147.32 107.95 0)
       (effects (font (size 1.27 1.27)) hide)
     )
@@
       (project "drip-irrigation-sys-cc"
         (path "/41708c1e-19b2-4374-83f2-108076d82b45/202a1cab-a33b-4ef0-945c-8042c7ebf8be"
-          (reference "#PWR012") (unit 1)
+          (reference "#PWR041") (unit 1)
         )
       )
@@
   (symbol (lib_id "Device:R") (at 116.84 62.23 90) (unit 1)
     (in_bom yes) (on_board yes) (dnp no) (fields_autoplaced)
-    (property "Reference" "R7" (at 116.84 55.88 90)
+    (property "Reference" "R17" (at 116.84 55.88 90)
       (effects (font (size 1.27 1.27)))
     )
@@
       (project "drip-irrigation-sys-cc"
         (path "/41708c1e-19b2-4374-83f2-108076d82b45/202a1cab-a33b-4ef0-945c-8042c7ebf8be"
-          (reference "R7") (unit 1)
+          (reference "R17") (unit 1)
         )
       )
@@
   (symbol (lib_id "Device:C") (at 129.54 62.23 90) (unit 1)
     (in_bom yes) (on_board yes) (dnp no) (fields_autoplaced)
-    (property "Reference" "C14" (at 129.54 54.61 90)
+    (property "Reference" "C21" (at 129.54 54.61 90)
       (effects (font (size 1.27 1.27)))
     )
@@
       (effects (font (size 1.27 1.27)))
     )
-    (property "Footprint" "Capacitor_SMD:C_0201_0603Metric" (at 133.35 61.2648 0)
+    (property "Footprint" "Capacitor_SMD:C_0805_2012Metric" (at 133.35 61.2648 0)
       (effects (font (size 1.27 1.27)) hide)
     )
@@
       (effects (font (size 1.27 1.27)) hide)
     )
-    (property "Digikey" "490-3167-2-ND" (at 129.54 62.23 0)
+    (property "Digikey" "" (at 129.54 62.23 0)
       (effects (font (size 1.27 1.27)) hide)
     )
@@
       (project "drip-irrigation-sys-cc"
         (path "/41708c1e-19b2-4374-83f2-108076d82b45/202a1cab-a33b-4ef0-945c-8042c7ebf8be"
-          (reference "C14") (unit 1)
+          (reference "C21") (unit 1)
         )
       )
@@
       (effects (font (size 1.27 1.27) italic) hide)
     )
+    (property "Digikey" "MMBT3904TPMSTR-ND" (at 138.43 62.23 0)
+      (effects (font (size 1.27 1.27)) hide)
+    )
     (pin "1")

Commit message: PCB düzenlemesi yapıldı.
Parts:
- removed K1: Relay_SPDT, Relay_THT:Relay_SPDT_Omron-G5LE-1, symbol Relay:Relay_SPDT
- added K2: G5LE-1 DC5, RELAY_G5LE-1 DC5_OMR, symbol drip-irrigation-sys-cc:G5LE-1_DC5
Connections:
- net COM: now also K2.1
- net GND: now also K2.2
- net NC: now also K2.4
- net NO: now also K2.3
- net at Q1.2: now also K2.5
Changed lines of the file:
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@@
     (stroke (width 0) (type default))
   )
-  (wire (pts (xy 157.48 102.87) (xy 177.8 102.87))
+  (wire (pts (xy 110.49 90.17) (xy 107.95 90.17))
     (stroke (width 0) (type default))
   )
-  (wire (pts (xy 160.02 85.09) (xy 160.02 82.55))
+  (wire (pts (xy 146.05 67.31) (xy 146.05 95.25))
     (stroke (width 0) (type default))
   )
-  (wire (pts (xy 157.48 100.33) (xy 157.48 102.87))
+  (wire (pts (xy 133.985 100.33) (xy 138.43 100.33))
     (stroke (width 0) (type default))
   )
-  (wire (pts (xy 154.94 85.09) (xy 154.94 80.01))
-    (stroke (width 0) (type default))
-  )
-  (wire (pts (xy 146.05 67.31) (xy 146.05 85.09))
-    (stroke (width 0) (type default))
-  )
-  (wire (pts (xy 160.02 82.55) (xy 177.8 82.55))
+  (wire (pts (xy 110.49 100.33) (xy 107.95 100.33))
     (stroke (width 0) (type default))
   )
@@
     (stroke (width 0) (type default))
   )
-  (wire (pts (xy 146.05 85.09) (xy 147.32 85.09))
-    (stroke (width 0) (type default))
-  )
-  (wire (pts (xy 147.32 101.6) (xy 147.32 100.33))
+  (wire (pts (xy 109.22 95.25) (xy 110.49 95.25))
     (stroke (width 0) (type default))
   )
@@
     (stroke (width 0) (type default))
   )
-  (wire (pts (xy 154.94 80.01) (xy 177.8 80.01))
+  (wire (pts (xy 133.985 95.25) (xy 146.05 95.25))
     (stroke (width 0) (type default))
   )
-  (hierarchical_label "COM" (shape input) (at 177.8 102.87 0) (fields_autoplaced)
-    (effects (font (size 1.27 1.27)) (justify left))
+  (hierarchical_label "COM" (shape input) (at 107.95 90.17 180) (fields_autoplaced)
+    (effects (font (size 1.27 1.27)) (justify right))
   )
-  (hierarchical_label "NO" (shape output) (at 177.8 82.55 0) (fields_autoplaced)
-    (effects (font (size 1.27 1.27)) (justify left))
+  (hierarchical_label "NO" (shape output) (at 107.95 100.33 180) (fields_autoplaced)
+    (effects (font (size 1.27 1.27)) (justify right))
   )
   (hierarchical_label "MCU_RELAY_PIN" (shape output) (at 104.14 62.23 180) (fields_autoplaced)
     (effects (font (size 1.27 1.27)) (justify right))
   )
-  (hierarchical_label "NC" (shape output) (at 177.8 80.01 0) (fields_autoplaced)
+  (hierarchical_label "NC" (shape output) (at 138.43 100.33 0) (fields_autoplaced)
     (effects (font (size 1.27 1.27)) (justify left))
   )
@@
     )
   )
-  (symbol (lib_id "power:GND") (at 147.32 101.6 0) (unit 1)
+  (symbol (lib_id "power:GND") (at 109.22 95.25 270) (unit 1)
     (in_bom yes) (on_board yes) (dnp no) (fields_autoplaced)
-    (property "Reference" "#PWR041" (at 147.32 107.95 0)
+    (property "Reference" "#PWR041" (at 102.87 95.25 0)
       (effects (font (size 1.27 1.27)) hide)
     )
-    (property "Value" "GND" (at 147.32 106.68 0)
+    (property "Value" "GND" (at 104.14 95.25 0)
       (effects (font (size 1.27 1.27)))
     )
-    (property "Footprint" "" (at 147.32 101.6 0)
+    (property "Footprint" "" (at 109.22 95.25 0)
       (effects (font (size 1.27 1.27)) hide)
     )
-    (property "Datasheet" "" (at 147.32 101.6 0)
+    (property "Datasheet" "" (at 109.22 95.25 0)
       (effects (font (size 1.27 1.27)) hide)
     )
@@
         (path "/41708c1e-19b2-4374-83f2-108076d82b45/202a1cab-a33b-4ef0-945c-8042c7ebf8be"
           (reference "#PWR041") (unit 1)
+        )
+      )
+    )
+  )
+  (symbol (lib_id "drip-irrigation-sys-cc:G5LE-1_DC5") (at 110.49 90.17 0) (unit 1)
+    (in_bom yes) (on_board yes) (dnp no) (fields_autoplaced)
+    (property "Reference" "K2" (at 122.2375 82.55 0)
+      (effects (font (size 1.524 1.524)))
+    )
+    (property "Value" "G5LE-1 DC5" (at 122.2375 85.09 0)
+      (effects (font (size 1.524 1.524)))
+    )
+    (property "Footprint" "RELAY_G5LE-1 DC5_OMR" (at 110.49 90.17 0)
+      (effects (font (size 1.27 1.27) italic) hide)
+    )
+    (property "Datasheet" "G5LE-1 DC5" (at 110.49 90.17 0)
+      (effects (font (size 1.27 1.27) italic) hide)
+    )
+    (pin "1")
+    (pin "2")
+    (pin "3")
+    (pin "4")
+    (pin "5")
+    (instances
+      (project "drip-irrigation-sys-cc"
+        (path "/41708c1e-19b2-4374-83f2-108076d82b45/202a1cab-a33b-4ef0-945c-8042c7ebf8be"
+          (reference "K2") (unit 1)
         )
       )
@@
         )
       )
-    )
-  )
-  (symbol (lib_id "Relay:Relay_SPDT") (at 152.4 92.71 0) (unit 1)
-    (in_bom yes) (on_board yes) (dnp no) (fields_autoplaced)
-    (property "Reference" "K1" (at 163.83 91.44 0)
-      (effects (font (size 1.27 1.27)) (justify left))
-    )
-    (property "Value" "Relay_SPDT" (at 163.83 93.98 0)
-      (effects (font (size 1.27 1.27)) (justify left))
-    )
-    (property "Footprint" "Relay_THT:Relay_SPDT_Omron-G5LE-1" (at 163.83 93.98 0)
-      (effects (font (size 1.27 1.27)) (justify left) hide)
-    )
-    (property "Datasheet" "~" (at 152.4 92.71 0)
-      (effects (font (size 1.27 1.27)) hide)
-    )
-    (property "Digikey" "Z3672-ND" (at 152.4 92.71 0)
-      (effects (font (size 1.27 1.27)) hide)
-    )
-    (pin "11")
-    (pin "12")
-    (pin "14")
-    (pin "A1")
-    (pin "A2")
-    (instances
-      (project "drip-irrigation-sys-cc"
-        (path "/41708c1e-19b2-4374-83f2-108076d82b45/202a1cab-a33b-4ef0-945c-8042c7ebf8be"
-          (reference "K1") (unit 1)
-        )
-      )
