File: hardware/relay.kicad_sch (KiCad schematic)
At the start: 4 parts, among them K2 G5LE-1 DC5, Q1 MMBT3904-TP

Commit message: PCB düzenleme.
Parts:
- C21: Digikey (none) -> 3372-0805B104K500BDTR-ND
- K2: Digikey (none) -> Z1014-ND
Changed lines of the file:
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@@
       (effects (font (size 1.27 1.27) italic) hide)
+    )
+    (property "Digikey" "Z1014-ND" (at 110.49 90.17 0)
+      (effects (font (size 1.27 1.27)) hide)
     )
     (pin "1")
@@
       (effects (font (size 1.27 1.27)) hide)
     )
-    (property "Digikey" "" (at 129.54 62.23 0)
+    (property "Digikey" "3372-0805B104K500BDTR-ND" (at 129.54 62.23 0)
       (effects (font (size 1.27 1.27)) hide)
     )
