File: hardware/drip-irrigation-sys-cc.kicad_pcb (KiCad board)
At the start: 2 copper layers, 108 parts, among them IC1 DALC208SC6, J1 PWR, J10 JAE_SIM_Card_SF72S006, J11 U.FL-R-SMT-1_10_, J2 USB_A, J3 PRESSURE_SENSOR, J4 Conn_02x01, J5 RELAY, J6 Conn_01x02_Pin, J7 Conn_01x04_Pin, J8 Conn_02x01, J9 Conn_02x06_Top_Bottom, K2 G5LE-1-VD-DC12, Q1 MMBT3904-TP, SW1 BTN_DEACTIVE, SW2 BTN_IO, SW3 BTN_ACTIVE, SW4 BTN_DEACTIVE, SW5 BTN_DEACTIVE, U1 STM32F103RCTx, U2 MAX3222EWN_T, U3 Max3075EESA, U4 MIC5504-3.3YM5-TR, U5 LM2576-5.0WU-TR, Y1 8MHZ, Y2 32KHZ

Commit message: PCB düzenlemesi yapıldı.
Parts:
- K2: value G5LE-1-VD-DC12 -> G5LE-1 DC5; footprint Relay_THT:Relay_SPDT_Omron-G5LE-1 -> drip-irrigation-sys-cc:RELAY_G5LE-1 DC5_OMR
- U2: footprint drip-irrigation-sys-cc:SOP65P640X120-20N -> drip-irrigation-sys-cc:MAX3222EWN+T
- moved C20 209.9 mm to (273.1, 47.5)
- moved J8 209.9 mm to (266.1, 42.0)
- moved R14 209.9 mm to (275.5, 37.9)
- moved R15 209.9 mm to (275.5, 40.4)
- moved R16 209.9 mm to (275.5, 42.9)
- moved U3 209.9 mm to (266.7, 49.2)
- moved H1 183.6 mm to (200.0, 20.6)
- moved H2 177.8 mm to (200.0, 27.1)
- moved H3 172.4 mm to (200.0, 33.7)
- moved H4 167.5 mm to (200.0, 40.2)
- moved C1 162.1 mm to (194.1, 47.8), turned to 0 degrees
- moved C28 152.3 mm to (231.8, 22.3)
- moved C29 152.3 mm to (231.8, 32.4)
- moved C30 152.3 mm to (253.8, 38.9)
- moved C31 152.3 mm to (253.8, 41.9)
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Connections:
- B1 pad 1: +5V -> GND
- C1 pad 2: +5V -> GND
- C10 pad 1: +5V -> GND
- C11 pad 2: +5V -> GND
- C12 pad 1: +5V -> GND
- C13 pad 2: +5V -> GND
- C14 pad 1: +5V -> GND
- C17 pad 2: +5V -> GND
- C18 pad 2: +5V -> GND
- C19 pad 2: +5V -> GND
- C2 pad 1: +5V -> GND
- C20 pad 2: +5V -> GND
- C23 pad 2: +5V -> GND
- C24 pad 2: +5V -> GND
- C25 pad 2: +5V -> GND
- C26 pad 2: +5V -> GND
- C27 pad 2: +5V -> GND
- C28 pad 2: +5V -> GND
- C29 pad 2: +5V -> GND
- C3 pad 1: +5V -> GND
- C30 pad 2: +5V -> GND
- C31 pad 2: +5V -> GND
- C32 pad 2: +5V -> GND
- C33 pad 2: +5V -> GND
- C34 pad 2: +5V -> GND
- C35 pad 2: +5V -> GND
- C36 pad 2: +5V -> GND
- C37 pad 2: +5V -> GND
- C38 pad 2: +5V -> GND
- C39 pad 2: +5V -> GND
- C4 pad 1: +5V -> GND
- C5 pad 2: +5V -> GND
- C6 pad 2: +5V -> GND
- C7 pad 2: +5V -> GND
- C8 pad 1: +5V -> GND
- C9 pad 1: +5V -> GND
- D1 pad 1: +5V -> GND
- D2 pad 1: +5V -> GND
- D3 pad 1: +5V -> GND
- D5 pad 2: +5V -> GND
- D7 pad 2: +5V -> GND
- D8 pad 1: +5V -> GND
- IC1 pad 5: +5V -> GND
- J10 pad C5: +5V -> GND
- J11 pad 1: +5V -> GND
- J2 pad 4: +5V -> GND
- J3 pad 3: +5V -> GND
- J7 pad 4: +5V -> GND
- J9 pad 11: +5V -> GND
- J9 pad 12: +5V -> GND
- K2 pad 2: +5V -> GND
- L1 pad 4: +5V -> GND
- R10 pad 2: +5V -> GND
- R13 pad 2: +5V -> GND
- R14 pad 2: +5V -> GND
- R16 pad 2: +5V -> GND
- SW1 pad 2: +5V -> GND
- SW2 pad 2: +5V -> GND
- SW3 pad 2: +5V -> GND
- SW4 pad 2: +5V -> GND
- SW5 pad 2: +5V -> GND
- U1 pad 12: +5V -> GND
- U1 pad 18: +5V -> GND
- U1 pad 31: +5V -> GND
- U1 pad 47: +5V -> GND
- U1 pad 63: +5V -> GND
- U2 pad 1: +5V -> GND
- U2 pad 16: +5V -> GND
- U3 pad 5: +5V -> GND
- U4 pad 2: +5V -> GND
- U5 pad 3: +5V -> GND
- U5 pad 5: +5V -> GND
- U6 pad 1: +5V -> GND
- U6 pad 10: +5V -> GND
- U6 pad 27: +5V -> GND
- U6 pad 34: +5V -> GND
- U6 pad 36: +5V -> GND
- U6 pad 37: +5V -> GND
- U6 pad 40: +5V -> GND
- U6 pad 41: +5V -> GND
Routing:
- net +5V: track 240.5 -> 0.00 mm
- net Net-(D5-K): track 51.0 -> 0.00 mm
- net /Relay/NO: track 0.00 -> 50.5 mm
- net Net-(D4-K): track 46.4 -> 0.00 mm, vias 3 -> 0
- net /Power/PWR_GND: track 43.1 -> 0.00 mm
- net /EXP/SPI_MISO: track 0.00 -> 37.3 mm
- net /Relay/NC: track 0.00 -> 37.3 mm
- net /MCU/BTN_DEACTIVATE: track 2.03 -> 31.6 mm
- net /EXP/USART3_TX: track 0.00 -> 29.6 mm, vias 0 -> 2
- net /EXP/I2C_SDL: track 0.00 -> 28.9 mm, vias 0 -> 2
- net Net-(K2-Pad5): track 0.00 -> 27.3 mm
- net /EXP/SPI_SCK: track 0.00 -> 23.7 mm, vias 0 -> 4
- net +12V: track 22.8 -> 0.00 mm
- net /Relay/COM: track 0.00 -> 22.6 mm, vias 0 -> 2
- net /EXP/USAR3_RX: track 0.00 -> 22.2 mm, vias 0 -> 2
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Other:
- board outline added: 126.5 x 126.5 mm

Commit message: PCB düzenlemesi.
Parts:
- C22, C23: footprint Capacitor_Tantalum_SMD:CP_EIA-1608-08_AVX-J -> Capacitor_SMD:C_0805_2012Metric
- C30: footprint Capacitor_SMD:C_0805_2012Metric -> Capacitor_Tantalum_SMD:CP_EIA-6032-15_Kemet-U
- moved C36 240.3 mm to (35.2, 131.6), turned to 180 degrees
- moved J10 232.5 mm to (27.6, 123.2)
- moved C35 231.2 mm to (42.1, 121.1), turned to -90 degrees
- moved C37 230.7 mm to (44.9, 132.7)
- moved C38 228.4 mm to (44.9, 129.5)
- moved IC1 226.7 mm to (39.6, 127.6)
- moved C39 226.3 mm to (44.9, 126.5)
- moved C32 222.4 mm to (39.1, 103.1), turned to 180 degrees
- moved R21 214.0 mm to (35.2, 128.5)
- moved U6 213.8 mm to (58.2, 126.6)
- moved R20 213.3 mm to (39.6, 132.2)
- moved C31 209.7 mm to (53.5, 104.1), turned to 180 degrees
- moved R22 207.7 mm to (37.1, 121.0), turned to 90 degrees
- moved C29 207.5 mm to (39.1, 109.3), turned to 180 degrees
- moved C30 207.0 mm to (55.8, 99.3), turned to 180 degrees
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Connections:
- R24 pad 1: /GSM_Module/NETLIGHT -> /GSM_Module/Net_light
Routing:
- net GND: track 0.00 -> 719.3 mm, vias 0 -> 59
- net +5V: track 0.00 -> 250.8 mm, vias 0 -> 20
- net +3.3V: track 17.4 -> 128.0 mm, vias 2 -> 11
- net /GSM_Module/4v: track 0.00 -> 70.9 mm, vias 0 -> 4
- net /MCU/USB_DM: track 0.00 -> 67.8 mm, vias 0 -> 2
- net /MCU/USB_DP: track 0.00 -> 66.2 mm, vias 0 -> 2
- net /ADC/MCU_ADC: track 3.58 -> 68.3 mm, vias 0 -> 2
- net /MCU/USART2_RX: track 0.00 -> 51.9 mm, vias 0 -> 2
- net /MCU/USART2_TX: track 0.00 -> 49.7 mm, vias 0 -> 2
- net +12V: track 0.00 -> 48.9 mm
- net /GSM_Module/SIM_VDD: track 0.00 -> 45.8 mm, vias 0 -> 4
- net +3V3: track 0.00 -> 44.3 mm, vias 0 -> 4
- net Net-(J10-RST): track 0.00 -> 34.2 mm
- net Net-(D5-K): track 0.00 -> 33.1 mm
- net Net-(U1-VBAT): track 0.00 -> 32.8 mm, vias 0 -> 2
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