File: hardware/gsm_module.kicad_sch (KiCad schematic)
At the start: 30 parts, among them IC1 DALC208SC6, J1 JAE_SIM_Card_SF72S006

Commit message: Kicad şema düzenlemesi yapıldı.
Parts:
- C12: footprint (none) -> Capacitor_Tantalum_SMD:CP_EIA-6032-20_AVX-F
- D4: footprint (none) -> drip-irrigation-sys-cc:DO-201AD_STM
- IC1: DigiKey 497-2525-2-ND -> (none); Digikey (none) -> 497-2525-2-ND
- J1: DigiKey 670-2967-2-ND -> (none)
- R10: footprint (none) -> Resistor_SMD:R_2512_6332Metric
Other:
- note added: "Supports up to 3A"

Commit message: Kicad şema düzenlemesi yapıldı.
Parts:
- C30: renamed from C1; Digikey (none) -> 399-C0805C330K5GAC7800TR-ND
- C31: renamed from C2; Digikey (none) -> 732-8077-2-ND
- C36: renamed from C11; Digikey (none) -> 399-C0805C330K5GAC7800TR-ND
- C37: renamed from C4; Digikey (none) -> 399-C0805C330K5GAC7800TR-ND
- C38: renamed from C5; Digikey (none) -> 399-C0805C330K5GAC7800TR-ND
- R20: renamed from R2; Digikey (none) -> 2577-AR03DTC1502TR-ND
- renumbered ANT1 to ANT2, C10 to C32, C6 to C33, C7 to C34, C3 to C35, C12 to C39, C8 to C40, C9 to C41, D4 to D5, D1 to D6, IC1 to IC2, J1 to J6, R1 to R19, R10 to R21, R3 to R22, R4 to R23, R6 to R24, R8 to R25, R7 to R26, R5 to R27, R9 to R28, S1 to S3, S2 to S4, U1 to U6

Commit message: Kicad şema düzenlemesi yapıldı.
Parts:
- removed ANT2: ACA-5036-A2-CC-S, mergened_footprints:ACA-5036-A2-CC-S, symbol mergened_symbols:ACA-5036-A2-CC-S
- removed C30, C36, C37, C38: 33pF, Capacitor_SMD:C_0805_2012Metric, symbol Device:C
- removed C31: 33nf, Capacitor_SMD:C_0805_2012Metric, symbol Device:C
- removed C32: 100uF, Capacitor_SMD:CP_Elec_8x10.5, symbol Device:C_Polarized_Small_US
- removed C33: 470uF, Capacitor_SMD:CP_Elec_8x10.5, symbol Device:C_Polarized_Small_US
- removed C34: 0.1uF, Capacitor_SMD:C_0805_2012Metric, symbol Device:C
- removed C35: 100uf, drip-irrigation-sys-cc:CAP_WCAP-ASLI_06p3X05p5_WRE, symbol Device:C
- removed C39: Tantalum 100uf, Capacitor_Tantalum_SMD:CP_EIA-6032-20_AVX-F, symbol Device:C
- removed C40, C41: ~, Capacitor_SMD:C_0805_2012Metric, symbol Device:C
- removed D5: D, drip-irrigation-sys-cc:DO-201AD_STM, symbol Device:D
- removed D6: LED, LED_SMD:LED_0805_2012Metric, symbol Device:LED
- removed IC2: DALC208SC6, mergened_footprints:DALC208SC6, symbol DALC208SC6:DALC208SC6
- removed J6: JAE_SIM_Card_SF72S006, Connector_JAE:JAE_SIM_Card_SF72S006, symbol Connector:JAE_SIM_Card_SF72S006
- removed R19, R22, R23: 22R, Resistor_SMD:R_0603_1608Metric, symbol Device:R
- removed R20: 15K, Resistor_SMD:R_0603_1608Metric, symbol Device:R
- removed R21: 100mOhm, Resistor_SMD:R_2512_6332Metric, symbol Device:R
- removed R24, R25: 0, Resistor_SMD:R_0603_1608Metric, symbol Device:R
- removed R26, R27, R28: 1K, Resistor_SMD:R_0603_1608Metric, symbol Device:R
- removed S3, S4: SKRPABE010, symbol Button_SKRPABE010:SKRPABE010
- removed U6: ~, mergened_footprints:MG2608, symbol mergened_symbols:mg2608
- added ANT?: ACA-5036-A2-CC-S, drip-irrigation-sys-cc:ACA-5036-A2-CC-S, symbol mergened_symbols:ACA-5036-A2-CC-S
- added C?: 470uF, Capacitor_SMD:CP_Elec_8x10.5, symbol Device:C_Polarized_Small_US
- added C?: 0.1uF, Capacitor_SMD:C_0805_2012Metric, symbol Device:C
- added C? (x4): 33pF, Capacitor_SMD:C_0805_2012Metric, symbol Device:C_Small
- added C?: 100uF, Capacitor_SMD:CP_Elec_8x10.5, symbol Device:C_Polarized_Small_US
- added C? (x2): ~, Capacitor_SMD:C_0805_2012Metric, symbol Device:C
- added C?: 100uF, Capacitor_SMD:C_0805_2012Metric, symbol Device:C_Small
- added C?: 33pF, Capacitor_SMD:C_0805_2012Metric, symbol Device:C
- added C?: 1uF, Capacitor_SMD:C_0805_2012Metric, symbol Device:C_Small
- added D7: D_Zener, drip-irrigation-sys-cc:SMB-2_4P60X3P95_ONS, symbol Device:D_Zener
- added D?: D, Diode_SMD:D_SOD-123F, symbol Device:D
- added D?: LED, LED_SMD:LED_0805_2012Metric, symbol Device:LED
- added IC?: DALC208SC6, drip-irrigation-sys-cc:SOT23-6L_STM, symbol DALC208SC6:DALC208SC6
- added J?: JAE_SIM_Card_SF72S006, Connector_JAE:JAE_SIM_Card_SF72S006, symbol Connector:JAE_SIM_Card_SF72S006
- added R? (x3): 22R, Resistor_SMD:R_0603_1608Metric, symbol Device:R_Small
- added R? (x3): 1K, Resistor_SMD:R_0603_1608Metric, symbol Device:R_Small
- added R?: 15K, Resistor_SMD:R_0603_1608Metric, symbol Device:R_Small
- added R? (x2): 0R, Resistor_SMD:R_0603_1608Metric, symbol Device:R
- added S? (x2): SKRPABE010, drip-irrigation-sys-cc:SW_PTS636_CNK, symbol Button_SKRPABE010:SKRPABE010
- added U?: ~, drip-irrigation-sys-cc:MG2608, symbol mergened_symbols:mg2608
Connections:
- net 4v: now also C?.1, C?.1, C?.1, C?.1, C?.1, D7.1 (K), D?.1 (K), R?.1, U?.42 (VBAT), U?.43 (VBAT)
- net GND: now also ANT?.GND1, ANT?.GND2, C?.2, C?.2, C?.2, C?.2, C?.2, C?.2, C?.2, C?.2, C?.2, C?.2, C?.2, C?.2, D7.2 (A), D?.1 (K), IC?.5 (REF_1), J?.C5 (GND), S?., S?., S?.2, S?.2, U?.1 (GND), U?.10 (GND), U?.27 (GND), U?.34 (GND), U?.36 (GND), U?.37 (GND), U?.40 (GND), U?.41 (GND)
- net Net_light: now also U?.16 (NETL_LIGHT)
- net PWRKEY: now also R?.1, U?.7 (PWRKEY)
- net REST: now also R?.1, U?.26 (REST)
- net SIM_CLK: now also C?.1, IC?.3 (I/O_2), R?.2, U?.13 (SIM_CLK)
- net SIM_DATA: now also C?.1, IC?.1 (I/O_1), R?.2, R?.2, U?.11 (SIM_DATA)
- new net: ANT?.FEED, C?.1, R?.1
- new net: J?.C2 (RST), R?.1
- new net: D?.2 (A), R?.2
- new net: J?.C3 (CLK), R?.1
- new net: J?.C7 (I/O), R?.1
- new net: R?.2, S?., S?.4 (x2)
- new net: C?.1, R?.1, R?.2
- new net 5V_Input: D?.2 (A)
- new net NETLIGHT: R?.1
- new net RF_ANT: R?.2, U?.35 (RF_ANT)
- new net SIM_RST: C?.1, IC?.4 (I/O_3), R?.2, U?.12 (SIM_RST)
- new net SIM_VDD: C?.1, C?.1, IC?.6 (I/O_4), J?.C1 (VCC), U?.14 (SIM_VDD)
- new net UART_RX: U?.17 (UART1_RXD)
- new net UART_TX: U?.18 (UART1_TXD)
- no-connect marks 0 -> 23
Other:
- note added: "ANTENNA"
- note added: "DECOUPLING"
- note added: "POWER Supports up to 3A"
- note added: "Tantalum"
- note removed: "Supports up to 3A"

Commit message: Kicad şema düzenlemesi.
Parts:
- removed ANT?: ACA-5036-A2-CC-S, drip-irrigation-sys-cc:ACA-5036-A2-CC-S, symbol mergened_symbols:ACA-5036-A2-CC-S
- added J11: U.FL-R-SMT-1_10_, drip-irrigation-sys-cc:HRS_U.FL-R-SMT-1_10_, symbol drip-irrigation-sys-cc:U.FL-R-SMT-1_10_
- S? (x2): Digikey (none) -> CKN12319-2-ND
Connections:
- net GND: now also J11.1
- net at C?.1, R?.1: now also J11.2
Changed lines of the file:
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@@
   (junction (at 35.306 49.276) (diameter 0) (color 0 0 0 0)
-  )
-  (junction (at 105.918 28.956) (diameter 0) (color 0 0 0 0)
   )
   (junction (at 41.148 49.276) (diameter 0) (color 0 0 0 0)
@@
     (stroke (width 0) (type default))
   )
-  (wire (pts (xy 105.918 26.416) (xy 105.918 28.956))
-    (stroke (width 0) (type default))
-  )
   (wire (pts (xy 241.808 143.002) (xy 241.808 146.558))
     (stroke (width 0) (type default))
@@
     (stroke (width 0) (type default))
   )
+  (wire (pts (xy 108.4144 23.876) (xy 108.4144 23.8716))
+    (stroke (width 0) (type default))
+  )
   (wire (pts (xy 149.606 126.492) (xy 156.972 126.492))
     (stroke (width 0) (type default))
@@
     (stroke (width 0) (type default))
   )
-  (wire (pts (xy 87.63 23.876) (xy 105.918 23.876))
+  (wire (pts (xy 87.63 23.876) (xy 108.4144 23.876))
     (stroke (width 0) (type default))
   )
@@
     (stroke (width 0) (type default))
   )
-  (wire (pts (xy 105.918 30.988) (xy 105.918 28.956))
+  (wire (pts (xy 105.918 26.416) (xy 105.918 30.988))
     (stroke (width 0) (type default))
   )
@@
   )
   (wire (pts (xy 142.748 107.696) (xy 165.862 107.696))
+    (stroke (width 0) (type default))
+  )
+  (wire (pts (xy 108.4144 26.416) (xy 108.4144 26.4116))
+    (stroke (width 0) (type default))
+  )
+  (wire (pts (xy 105.918 26.416) (xy 108.4144 26.416))
     (stroke (width 0) (type default))
   )
@@
     )
   )
-  (symbol (lib_id "mergened_symbols:ACA-5036-A2-CC-S") (at 108.458 26.416 0) (unit 1)
-    (in_bom yes) (on_board yes) (dnp no)
-    (property "Reference" "ANT?" (at 116.332 24.892 0)
-      (effects (font (size 1.27 1.27)) (justify left))
-    )
-    (property "Value" "ACA-5036-A2-CC-S" (at 114.808 36.322 90)
-      (effects (font (size 1.27 1.27)) (justify left))
-    )
-    (property "Footprint" "drip-irrigation-sys-cc:ACA-5036-A2-CC-S" (at 108.458 26.416 0)
-      (effects (font (size 1.27 1.27)) (justify bottom) hide)
-    )
-    (property "Datasheet" "" (at 108.458 26.416 0)
-      (effects (font (size 1.27 1.27)) hide)
-    )
-    (property "MF" "" (at 108.458 26.416 0)
-      (effects (font (size 1.27 1.27)) (justify bottom) hide)
-    )
-    (property "Description" "\n" (at 108.458 26.416 0)
-      (effects (font (size 1.27 1.27)) (justify bottom) hide)
-    )
-    (property "Package" "" (at 108.458 26.416 0)
-      (effects (font (size 1.27 1.27)) (justify bottom) hide)
-    )
-    (property "Price" "" (at 108.458 26.416 0)
-      (effects (font (size 1.27 1.27)) (justify bottom) hide)
-    )
-    (property "SnapEDA_Link" "" (at 108.458 26.416 0)
-      (effects (font (size 1.27 1.27)) (justify bottom) hide)
-    )
-    (property "MP" "" (at 108.458 26.416 0)
-      (effects (font (size 1.27 1.27)) (justify bottom) hide)
-    )
-    (property "Availability" "" (at 108.458 26.416 0)
-      (effects (font (size 1.27 1.27)) (justify bottom) hide)
-    )
-    (property "Check_prices" "" (at 108.458 26.416 0)
-      (effects (font (size 1.27 1.27)) (justify bottom) hide)
-    )
-    (pin "FEED")
-    (pin "GND1")
-    (pin "GND2")
-    (instances
-      (project "gsm_module"
-        (path "/0ad6aedd-0f1e-4202-ba35-607319fc6ad5"
-          (reference "ANT?") (unit 1)
-        )
-      )
-      (project "sayac"
-        (path "/2dfe6560-cbb2-4256-b30d-a6bedc3b7f39/59250a6b-7d16-422b-88de-376c9d7ef623"
-          (reference "ANT?") (unit 1)
-        )
-      )
-      (project "drip-irrigation-sys-cc"
-        (path "/41708c1e-19b2-4374-83f2-108076d82b45/abe8ffe0-aaec-43ca-9ae1-9a3e5d5ac5b2"
-          (reference "ANT1") (unit 1)
-        )
-      )
-      (project "mg2608"
-        (path "/63a0379d-fc16-4019-b887-c3021204e6ee/c89e0226-58a3-4dd7-b4e1-774a42131142"
-          (reference "ANT?") (unit 1)
-        )
-      )
-    )
-  )
   (symbol (lib_id "Device:R_Small") (at 87.63 129.032 90) (unit 1)
     (in_bom yes) (on_board yes) (dnp no)
@@
       (effects (font (size 1.27 1.27)) (justify bottom) hide)
     )
+    (property "Digikey" "CKN12319-2-ND" (at 241.808 155.194 0)
+      (effects (font (size 1.27 1.27)) hide)
+    )
     (pin "")
     (pin "")
@@
     )
   )
+  (symbol (lib_id "drip-irrigation-sys-cc:U.FL-R-SMT-1_10_") (at 110.9544 23.8716 0) (unit 1)
+    (in_bom yes) (on_board yes) (dnp no) (fields_autoplaced)
+    (property "Reference" "J11" (at 113.4944 23.0461 0)
+      (effects (font (size 1.27 1.27)) (justify left))
+    )
+    (property "Value" "U.FL-R-SMT-1_10_" (at 113.4944 25.5861 0)
+      (effects (font (size 1.27 1.27)) (justify left))
+    )
+    (property "Footprint" "drip-irrigation-sys-cc:HRS_U.FL-R-SMT-1_10_" (at 110.9544 23.8716 0)
+      (effects (font (size 1.27 1.27)) (justify bottom) hide)
+    )
+    (property "Datasheet" "" (at 110.9544 23.8716 0)
+      (effects (font (size 1.27 1.27)) hide)
+    )
+    (property "DESCRIPTION" "U.FL Series 6 Ghz 50 Ohm Ultra-small SMT Coaxial Cable Receptacle" (at 110.9544 23.8716 0)
+      (effects (font (size 1.27 1.27)) (justify bottom) hide)
+    )
+    (property "PACKAGE" "None" (at 110.9544 23.8716 0)
+      (effects (font (size 1.27 1.27)) (justify bottom) hide)
+    )
+    (property "PRICE" "0.71 USD" (at 110.9544 23.8716 0)
+      (effects (font (size 1.27 1.27)) (justify bottom) hide)
+    )
+    (property "STANDARD" "Manufacturer Recommendation" (at 110.9544 23.8716 0)
+      (effects (font (size 1.27 1.27)) (justify bottom) hide)
+    )
+    (property "MP" "U.FL-R-SMT-1_10_" (at 110.9544 23.8716 0)
+      (effects (font (size 1.27 1.27)) (justify bottom) hide)
+    )
+    (property "AVAILABILITY" "Good" (at 110.9544 23.8716 0)
+      (effects (font (size 1.27 1.27)) (justify bottom) hide)
+    )
+    (property "MANUFACTURER" "Hirose" (at 110.9544 23.8716 0)
+      (effects (font (size 1.27 1.27)) (justify bottom) hide)
+    )
+    (pin "1")
+    (pin "2")
+    (instances
+      (project "drip-irrigation-sys-cc"
+        (path "/41708c1e-19b2-4374-83f2-108076d82b45/abe8ffe0-aaec-43ca-9ae1-9a3e5d5ac5b2"
+          (reference "J11") (unit 1)
+        )
+      )
+    )
+  )
   (symbol (lib_id "Button_SKRPABE010:SKRPABE010") (at 261.366 155.448 90) (unit 1)
     (in_bom yes) (on_board yes) (dnp no)
@@
       (effects (font (size 1.27 1.27)) (justify bottom) hide)
     )
+    (property "Digikey" "CKN12319-2-ND" (at 261.366 155.448 0)
+      (effects (font (size 1.27 1.27)) hide)
+    )
     (pin "")

Commit message: PCB düzenlemesi yapıldı.
Parts:
- removed S? (x2): SKRPABE010, drip-irrigation-sys-cc:SW_PTS636_CNK, symbol Button_SKRPABE010:SKRPABE010
- added SW1 (x2): BTN_DEACTIVE, SW_PTS636_CNK, symbol drip-irrigation-sys-cc:PTS636_SM50J_SMTR_LFS
Connections:
- net GND: now also SW1.2, SW1.2
- net at R?.2: now also SW1.1 (x2)

Commit message: PCB düzenlemesi.
Parts:
- C?: footprint Capacitor_SMD:C_0805_2012Metric -> Capacitor_Tantalum_SMD:CP_EIA-6032-15_Kemet-U; Digikey (none) -> TCKOJ107CT
Connections:
- net NETLIGHT is gone; now on net Net_light: R?.1
- no-connect marks 23 -> 27
Changed lines of the file:
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@@
   )
   (no_connect (at 106.426 105.156))
+  (no_connect (at 77.47 146.812))
   (no_connect (at 219.71 49.784))
   (no_connect (at 254 30.48))
   (no_connect (at 219.71 92.202))
+  (no_connect (at 77.47 141.732))
   (no_connect (at 264.414 61.468))
   (no_connect (at 219.71 45.212))
@@
   (no_connect (at 264.414 59.182))
   (no_connect (at 264.414 49.784))
+  (no_connect (at 77.47 144.272))
+  (no_connect (at 77.47 136.652))
   (wire (pts (xy 76.454 23.876) (xy 77.978 23.876))
     (stroke (width 0) (type default))
@@
     (effects (font (size 1.27 1.27)) (justify right bottom))
   )
+  (label "Net_light" (at 222.504 125.984 90) (fields_autoplaced)
+    (effects (font (size 1.27 1.27)) (justify left bottom))
+  )
   (label "RF_ANT" (at 57.404 23.876 0) (fields_autoplaced)
     (effects (font (size 1.27 1.27)) (justify left bottom))
@@
   (label "VIN" (at 17.78 22.86 0) (fields_autoplaced)
     (effects (font (size 1.27 1.27)) (justify left bottom))
-  )
-  (label "NETLIGHT" (at 222.504 125.984 270) (fields_autoplaced)
-    (effects (font (size 1.27 1.27)) (justify right bottom))
   )
   (label "PWRKEY" (at 261.366 125.984 270) (fields_autoplaced)
@@
       (effects (font (size 1.27 1.27)) (justify left))
     )
-    (property "Footprint" "Capacitor_SMD:C_0805_2012Metric" (at 35.56 27.94 0)
+    (property "Footprint" "Capacitor_Tantalum_SMD:CP_EIA-6032-15_Kemet-U" (at 35.56 27.94 0)
       (effects (font (size 1.27 1.27)) hide)
     )
@@
       (effects (font (size 1.27 1.27)) hide)
     )
+    (property "Digikey" "TCKOJ107CT" (at 35.56 27.94 0)
+      (effects (font (size 1.27 1.27)) hide)
+    )

Commit message: PCB düzenleme.
Parts:
- C?: Digikey (none) -> 2997-SRF10V471MJ102-ND
- C?: Digikey (none) -> 3372-0805B104K201DCTR-ND
- C? (x5): footprint Capacitor_SMD:C_0805_2012Metric -> Capacitor_SMD:C_0603_1608Metric; Digikey (none) -> 2571-GMC10CG330K100NTTR-ND
- C?: Digikey (none) -> 2997-SHT6.3V101M-F55-ND
- C?: Digikey (none) -> 3372-0805B105K100CCTR-ND
- D?: Digikey (none) -> 3372-0805YGBD008S01TR-ND
- R? (x3): Digikey (none) -> 311-22.0HRDKR-ND
- R?: Digikey (none) -> P15KDBDKR-ND
Changed lines of the file:
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@@
+      (effects (font (size 1.27 1.27)) hide)
+    )
+    (property "Digikey" "311-22.0HRDKR-ND" (at 87.63 129.032 0)
       (effects (font (size 1.27 1.27)) hide)
     )
@@
     )
     (property "Datasheet" "~" (at 28.448 54.61 0)
+      (effects (font (size 1.27 1.27)) hide)
+    )
+    (property "Digikey" "2997-SRF10V471MJ102-ND" (at 28.448 54.61 0)
       (effects (font (size 1.27 1.27)) hide)
     )
@@
       (effects (font (size 1.27 1.27)) hide)
     )
+    (property "Digikey" "P15KDBDKR-ND" (at 89.408 96.774 0)
+      (effects (font (size 1.27 1.27)) hide)
+    )
     (pin "1")
     (pin "2")
@@
       (effects (font (size 1.27 1.27)) hide)
     )
+    (property "Digikey" "3372-0805B104K201DCTR-ND" (at 41.148 54.356 0)
+      (effects (font (size 1.27 1.27)) hide)
+    )
     (pin "1")
     (pin "2")
@@
       (effects (font (size 1.27 1.27)) (justify left))
     )
-    (property "Footprint" "Capacitor_SMD:C_0805_2012Metric" (at 142.748 144.78 0)
+    (property "Footprint" "Capacitor_SMD:C_0603_1608Metric" (at 142.748 144.78 0)
       (effects (font (size 1.27 1.27)) hide)
     )
     (property "Datasheet" "~" (at 142.748 144.78 0)
+      (effects (font (size 1.27 1.27)) hide)
+    )
+    (property "Digikey" "2571-GMC10CG330K100NTTR-ND" (at 142.748 144.78 0)
       (effects (font (size 1.27 1.27)) hide)
     )
@@
       (effects (font (size 1.27 1.27)) hide)
     )
+    (property "Digikey" "311-22.0HRDKR-ND" (at 87.63 131.572 0)
+      (effects (font (size 1.27 1.27)) hide)
+    )
     (pin "1")
     (pin "2")
@@
       (effects (font (size 1.27 1.27)) hide)
     )
+    (property "Digikey" "2997-SHT6.3V101M-F55-ND" (at 18.288 54.864 0)
+      (effects (font (size 1.27 1.27)) hide)
+    )
     (pin "1")
     (pin "2")
@@
       (effects (font (size 1.27 1.27)) hide)
     )
+    (property "Digikey" "311-22.0HRDKR-ND" (at 87.63 139.192 0)
+      (effects (font (size 1.27 1.27)) hide)
+    )
     (pin "1")
     (pin "2")
@@
       (effects (font (size 1.27 1.27)) (justify left))
     )
-    (property "Footprint" "Capacitor_SMD:C_0805_2012Metric" (at 94.996 144.78 0)
+    (property "Footprint" "Capacitor_SMD:C_0603_1608Metric" (at 94.996 144.78 0)
       (effects (font (size 1.27 1.27)) hide)
     )
@@
       (effects (font (size 1.27 1.27)) hide)
     )
+    (property "Digikey" "2571-GMC10CG330K100NTTR-ND" (at 94.996 144.78 0)
+      (effects (font (size 1.27 1.27)) hide)
+    )
     (pin "1")
     (pin "2")
@@
       (effects (font (size 1.27 1.27)) (justify left))
     )
-    (property "Footprint" "Capacitor_SMD:C_0805_2012Metric" (at 50.4952 58.166 0)
+    (property "Footprint" "Capacitor_SMD:C_0603_1608Metric" (at 50.4952 58.166 0)
       (effects (font (size 1.27 1.27)) hide)
     )
     (property "Datasheet" "~" (at 49.53 54.356 0)
+      (effects (font (size 1.27 1.27)) hide)
+    )
+    (property "Digikey" "2571-GMC10CG330K100NTTR-ND" (at 49.53 54.356 0)
       (effects (font (size 1.27 1.27)) hide)
     )
@@
       (effects (font (size 1.27 1.27)) (justify left))
     )
-    (property "Footprint" "Capacitor_SMD:C_0805_2012Metric" (at 104.394 144.78 0)
+    (property "Footprint" "Capacitor_SMD:C_0603_1608Metric" (at 104.394 144.78 0)
       (effects (font (size 1.27 1.27)) hide)
     )
@@
       (effects (font (size 1.27 1.27)) hide)
     )
+    (property "Digikey" "2571-GMC10CG330K100NTTR-ND" (at 104.394 144.78 0)
+      (effects (font (size 1.27 1.27)) hide)
+    )
     (pin "1")
     (pin "2")
@@
     )
     (property "Datasheet" "~" (at 222.504 150.876 0)
+      (effects (font (size 1.27 1.27)) hide)
+    )
+    (property "Digikey" "3372-0805YGBD008S01TR-ND" (at 222.504 150.876 0)
       (effects (font (size 1.27 1.27)) hide)
     )
@@
       (effects (font (size 1.27 1.27)) hide)
     )
+    (property "Digikey" "3372-0805B105K100CCTR-ND" (at 156.972 144.78 0)
+      (effects (font (size 1.27 1.27)) hide)
+    )
     (pin "1")
     (pin "2")
@@
       (effects (font (size 1.27 1.27)) (justify left))
     )
-    (property "Footprint" "Capacitor_SMD:C_0805_2012Metric" (at 149.606 144.78 0)
+    (property "Footprint" "Capacitor_SMD:C_0603_1608Metric" (at 149.606 144.78 0)
       (effects (font (size 1.27 1.27)) hide)
     )
@@
       (effects (font (size 1.27 1.27)) hide)
     )
+    (property "Digikey" "2571-GMC10CG330K100NTTR-ND" (at 149.606 144.78 0)
+      (effects (font (size 1.27 1.27)) hide)
+    )
