File: hardware/mcu.kicad_sch (KiCad schematic)
At the start: 15 parts, among them J5 Conn_01x04_Pin, U4 STM32F103RCTx, Y1 8MHZ, Y2 32KHZ

Commit message: Kicad şema düzenlemesi yapıldı.
Parts:
- R12: footprint (none) -> Resistor_SMD:R_0402_1005Metric; Digikey (none) -> 1276-3431-2-ND
- R13: footprint (none) -> Resistor_SMD:R_1206_3216Metric; Digikey (none) -> 5440-FMF06FTHR010-LHMTR-ND
- Y1: footprint (none) -> drip-irrigation-sys-cc:XTAL_ABLS2_ABR; Digikey (none) -> 535-10212-2-ND
- Y2: footprint (none) -> drip-irrigation-sys-cc:XTAL_CM7V-T1A_MCX; Digikey (none) -> 2195-CM7V-T1A-32.768KHZ-7PF-20PPM-TB-QATR-ND
Other:
- moved on the sheet: C17, C18, Y2
Changed lines of the file:
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@@
   (junction (at 147.32 35.56) (diameter 0) (color 0 0 0 0)
   )
-  (junction (at 97.79 113.03) (diameter 0) (color 0 0 0 0)
+  (junction (at 110.49 113.03) (diameter 0) (color 0 0 0 0)
   )
   (junction (at 64.77 72.39) (diameter 0) (color 0 0 0 0)
   )
-  (junction (at 102.87 130.81) (diameter 0) (color 0 0 0 0)
+  (junction (at 115.57 130.81) (diameter 0) (color 0 0 0 0)
   )
   (junction (at 125.73 17.78) (diameter 0) (color 0 0 0 0)
@@
   (junction (at 143.51 138.43) (diameter 0) (color 0 0 0 0)
   )
-  (junction (at 107.95 113.03) (diameter 0) (color 0 0 0 0)
+  (junction (at 120.65 113.03) (diameter 0) (color 0 0 0 0)
   )
   (junction (at 93.98 22.86) (diameter 0) (color 0 0 0 0)
@@
     (stroke (width 0) (type default))
   )
-  (wire (pts (xy 97.79 100.33) (xy 124.46 100.33))
+  (wire (pts (xy 110.49 100.33) (xy 124.46 100.33))
     (stroke (width 0) (type default))
   )
@@
     (stroke (width 0) (type default))
   )
-  (wire (pts (xy 97.79 113.03) (xy 100.33 113.03))
+  (wire (pts (xy 110.49 113.03) (xy 113.03 113.03))
     (stroke (width 0) (type default))
   )
@@
     (stroke (width 0) (type default))
   )
-  (wire (pts (xy 97.79 118.11) (xy 97.79 113.03))
+  (wire (pts (xy 110.49 118.11) (xy 110.49 113.03))
     (stroke (width 0) (type default))
   )
@@
     (stroke (width 0) (type default))
   )
-  (wire (pts (xy 97.79 113.03) (xy 97.79 100.33))
+  (wire (pts (xy 110.49 113.03) (xy 110.49 100.33))
     (stroke (width 0) (type default))
   )
@@
     (stroke (width 0) (type default))
   )
-  (wire (pts (xy 107.95 113.03) (xy 107.95 102.87))
+  (wire (pts (xy 120.65 113.03) (xy 120.65 102.87))
     (stroke (width 0) (type default))
   )
@@
     (stroke (width 0) (type default))
   )
-  (wire (pts (xy 107.95 113.03) (xy 105.41 113.03))
-    (stroke (width 0) (type default))
-  )
-  (wire (pts (xy 107.95 130.81) (xy 107.95 123.19))
+  (wire (pts (xy 120.65 113.03) (xy 118.11 113.03))
+    (stroke (width 0) (type default))
+  )
+  (wire (pts (xy 120.65 130.81) (xy 120.65 123.19))
     (stroke (width 0) (type default))
   )
@@
     (stroke (width 0) (type default))
   )
-  (wire (pts (xy 107.95 102.87) (xy 124.46 102.87))
-    (stroke (width 0) (type default))
-  )
-  (wire (pts (xy 107.95 118.11) (xy 107.95 113.03))
+  (wire (pts (xy 120.65 102.87) (xy 124.46 102.87))
+    (stroke (width 0) (type default))
+  )
+  (wire (pts (xy 120.65 118.11) (xy 120.65 113.03))
     (stroke (width 0) (type default))
   )
@@
     (stroke (width 0) (type default))
   )
-  (wire (pts (xy 102.87 130.81) (xy 97.79 130.81))
+  (wire (pts (xy 115.57 130.81) (xy 110.49 130.81))
     (stroke (width 0) (type default))
   )
@@
     (stroke (width 0) (type default))
   )
-  (wire (pts (xy 102.87 130.81) (xy 107.95 130.81))
-    (stroke (width 0) (type default))
-  )
-  (wire (pts (xy 97.79 130.81) (xy 97.79 123.19))
+  (wire (pts (xy 115.57 130.81) (xy 120.65 130.81))
+    (stroke (width 0) (type default))
+  )
+  (wire (pts (xy 110.49 130.81) (xy 110.49 123.19))
     (stroke (width 0) (type default))
   )
@@
     )
   )
-  (symbol (lib_id "Device:C_Small") (at 97.79 120.65 0) (unit 1)
-    (in_bom yes) (on_board yes) (dnp no) (fields_autoplaced)
-    (property "Reference" "C17" (at 100.33 119.3863 0)
-      (effects (font (size 1.27 1.27)) (justify left))
-    )
-    (property "Value" "10pf" (at 100.33 121.9263 0)
-      (effects (font (size 1.27 1.27)) (justify left))
-    )
-    (property "Footprint" "Capacitor_SMD:C_0201_0603Metric" (at 97.79 120.65 0)
-      (effects (font (size 1.27 1.27)) hide)
-    )
-    (property "Datasheet" "~" (at 97.79 120.65 0)
-      (effects (font (size 1.27 1.27)) hide)
-    )
-    (property "Digikey" "490-8607-2-ND" (at 97.79 120.65 0)
+  (symbol (lib_id "Device:C_Small") (at 110.49 120.65 0) (unit 1)
+    (in_bom yes) (on_board yes) (dnp no) (fields_autoplaced)
+    (property "Reference" "C17" (at 113.03 119.3863 0)
+      (effects (font (size 1.27 1.27)) (justify left))
+    )
+    (property "Value" "10pf" (at 113.03 121.9263 0)
+      (effects (font (size 1.27 1.27)) (justify left))
+    )
+    (property "Footprint" "Capacitor_SMD:C_0201_0603Metric" (at 110.49 120.65 0)
+      (effects (font (size 1.27 1.27)) hide)
+    )
+    (property "Datasheet" "~" (at 110.49 120.65 0)
+      (effects (font (size 1.27 1.27)) hide)
+    )
+    (property "Digikey" "490-8607-2-ND" (at 110.49 120.65 0)
       (effects (font (size 1.27 1.27)) hide)
     )
@@
     )
   )
-  (symbol (lib_id "Device:C_Small") (at 107.95 120.65 0) (unit 1)
-    (in_bom yes) (on_board yes) (dnp no) (fields_autoplaced)
-    (property "Reference" "C18" (at 110.49 119.3863 0)
-      (effects (font (size 1.27 1.27)) (justify left))
-    )
-    (property "Value" "10pf" (at 110.49 121.9263 0)
-      (effects (font (size 1.27 1.27)) (justify left))
-    )
-    (property "Footprint" "Capacitor_SMD:C_0201_0603Metric" (at 107.95 120.65 0)
-      (effects (font (size 1.27 1.27)) hide)
-    )
-    (property "Datasheet" "~" (at 107.95 120.65 0)
-      (effects (font (size 1.27 1.27)) hide)
-    )
-    (property "Digikey" "490-8607-2-ND" (at 107.95 120.65 0)
+  (symbol (lib_id "Device:C_Small") (at 120.65 120.65 0) (unit 1)
+    (in_bom yes) (on_board yes) (dnp no) (fields_autoplaced)
+    (property "Reference" "C18" (at 123.19 119.3863 0)
+      (effects (font (size 1.27 1.27)) (justify left))
+    )
+    (property "Value" "10pf" (at 123.19 121.9263 0)
+      (effects (font (size 1.27 1.27)) (justify left))
+    )
+    (property "Footprint" "Capacitor_SMD:C_0201_0603Metric" (at 120.65 120.65 0)
+      (effects (font (size 1.27 1.27)) hide)
+    )
+    (property "Datasheet" "~" (at 120.65 120.65 0)
+      (effects (font (size 1.27 1.27)) hide)
+    )
+    (property "Digikey" "490-8607-2-ND" (at 120.65 120.65 0)
       (effects (font (size 1.27 1.27)) hide)
     )
@@
       (effects (font (size 1.27 1.27)))
     )
-    (property "Footprint" "" (at 59.69 72.39 0)
+    (property "Footprint" "drip-irrigation-sys-cc:XTAL_ABLS2_ABR" (at 59.69 72.39 0)
       (effects (font (size 1.27 1.27)) hide)
     )
     (property "Datasheet" "~" (at 59.69 72.39 0)
+      (effects (font (size 1.27 1.27)) hide)
+    )
+    (property "Digikey" "535-10212-2-ND" (at 59.69 72.39 0)
       (effects (font (size 1.27 1.27)) hide)
     )
@@
     )
   )
-  (symbol (lib_id "Device:Crystal_Small") (at 102.87 113.03 0) (unit 1)
-    (in_bom yes) (on_board yes) (dnp no) (fields_autoplaced)
-    (property "Reference" "Y2" (at 102.87 106.68 0)
-      (effects (font (size 1.27 1.27)))
-    )
-    (property "Value" "32KHZ" (at 102.87 109.22 0)
-      (effects (font (size 1.27 1.27)))
-    )
-    (property "Footprint" "" (at 102.87 113.03 0)
-      (effects (font (size 1.27 1.27)) hide)
-    )
-    (property "Datasheet" "~" (at 102.87 113.03 0)
+  (symbol (lib_id "Device:Crystal_Small") (at 115.57 113.03 0) (unit 1)
+    (in_bom yes) (on_board yes) (dnp no) (fields_autoplaced)
+    (property "Reference" "Y2" (at 115.57 106.68 0)
+      (effects (font (size 1.27 1.27)))
+    )
+    (property "Value" "32KHZ" (at 115.57 109.22 0)
+      (effects (font (size 1.27 1.27)))
+    )
+    (property "Footprint" "drip-irrigation-sys-cc:XTAL_CM7V-T1A_MCX" (at 115.57 113.03 0)
+      (effects (font (size 1.27 1.27)) hide)
+    )
+    (property "Datasheet" "~" (at 115.57 113.03 0)
+      (effects (font (size 1.27 1.27)) hide)
+    )
+    (property "Digikey" "2195-CM7V-T1A-32.768KHZ-7PF-20PPM-TB-QATR-ND" (at 115.57 113.03 0)
       (effects (font (size 1.27 1.27)) hide)
     )
@@
     )
   )
-  (symbol (lib_id "power:GND") (at 102.87 130.81 0) (unit 1)
-    (in_bom yes) (on_board yes) (dnp no) (fields_autoplaced)
-    (property "Reference" "#PWR025" (at 102.87 137.16 0)
-      (effects (font (size 1.27 1.27)) hide)
-    )
-    (property "Value" "GND" (at 102.87 135.89 0)
-      (effects (font (size 1.27 1.27)))
-    )
-    (property "Footprint" "" (at 102.87 130.81 0)
-      (effects (font (size 1.27 1.27)) hide)
-    )
-    (property "Datasheet" "" (at 102.87 130.81 0)
+  (symbol (lib_id "power:GND") (at 115.57 130.81 0) (unit 1)
+    (in_bom yes) (on_board yes) (dnp no) (fields_autoplaced)
+    (property "Reference" "#PWR025" (at 115.57 137.16 0)
+      (effects (font (size 1.27 1.27)) hide)
+    )
+    (property "Value" "GND" (at 115.57 135.89 0)
+      (effects (font (size 1.27 1.27)))
+    )
+    (property "Footprint" "" (at 115.57 130.81 0)
+      (effects (font (size 1.27 1.27)) hide)
+    )
+    (property "Datasheet" "" (at 115.57 130.81 0)
       (effects (font (size 1.27 1.27)) hide)
     )
@@
       (effects (font (size 1.27 1.27)))
     )
-    (property "Footprint" "" (at 59.69 62.738 90)
+    (property "Footprint" "Resistor_SMD:R_1206_3216Metric" (at 59.69 62.738 90)
       (effects (font (size 1.27 1.27)) hide)
     )
@@
       (effects (font (size 1.27 1.27)) hide)
     )
+    (property "Digikey" "5440-FMF06FTHR010-LHMTR-ND" (at 59.69 60.96 0)
+      (effects (font (size 1.27 1.27)) hide)
+    )
     (pin "1")
     (pin "2")
@@
       (effects (font (size 1.27 1.27)) (justify left))
     )
-    (property "Footprint" "" (at 111.252 39.37 90)
+    (property "Footprint" "Resistor_SMD:R_0402_1005Metric" (at 111.252 39.37 90)
       (effects (font (size 1.27 1.27)) hide)
     )
@@
       (effects (font (size 1.27 1.27)) hide)
     )
+    (property "Digikey" "1276-3431-2-ND" (at 113.03 39.37 0)
+      (effects (font (size 1.27 1.27)) hide)
+    )

Commit message: Kicad şema düzenlemesi yapıldı.
Parts:
- removed R13: 10mOhm, Resistor_SMD:R_1206_3216Metric, symbol Device:R
- added B1: BH-80B-1, BH-80B-1_ADM, symbol drip-irrigation-sys-cc:BH-80B-1
- added C5: 100nf, Capacitor_SMD:C_0805_2012Metric, symbol Device:C_Small
- added J6: Conn_01x02_Pin, Connector_PinHeader_2.54mm:PinHeader_1x02_P2.54mm_Vertical, symbol Connector:Conn_01x02_Pin
- added R10: 10K, Resistor_SMD:R_0603_1608Metric, symbol Device:R
- C10: renamed from C21; footprint Capacitor_SMD:C_0201_0603Metric -> Capacitor_SMD:C_0805_2012Metric; Digikey 490-3167-2-ND -> (none)
- C11: renamed from C17; footprint Capacitor_SMD:C_0201_0603Metric -> Capacitor_SMD:C_0805_2012Metric; Digikey 490-8607-2-ND -> (none)
- C12: renamed from C22; footprint Capacitor_SMD:C_0201_0603Metric -> Capacitor_SMD:C_0805_2012Metric; Digikey 490-3167-2-ND -> (none)
- C13: renamed from C18; footprint Capacitor_SMD:C_0201_0603Metric -> Capacitor_SMD:C_0805_2012Metric; Digikey 490-8607-2-ND -> (none)
- C14: renamed from C23; footprint Capacitor_SMD:C_1206_3216Metric -> Capacitor_SMD:C_0805_2012Metric; Digikey 5440-FN31X103K500PXGTR-ND -> (none)
- C6: renamed from C15; footprint Capacitor_SMD:C_0201_0603Metric -> Capacitor_SMD:C_0805_2012Metric; Digikey 490-8607-2-ND -> (none)
- C7: renamed from C16; footprint Capacitor_SMD:C_0201_0603Metric -> Capacitor_SMD:C_0805_2012Metric; Digikey 490-8607-2-ND -> (none)
- C8: renamed from C20; footprint Capacitor_SMD:C_0201_0603Metric -> Capacitor_SMD:C_0805_2012Metric; Digikey 490-3167-2-ND -> (none)
- C9: renamed from C13; footprint Capacitor_SMD:C_0201_0603Metric -> Capacitor_SMD:C_0805_2012Metric; Digikey 490-3167-2-ND -> (none)
- R11: renamed from R12; footprint Resistor_SMD:R_0402_1005Metric -> Resistor_SMD:R_0603_1608Metric; Digikey 1276-3431-2-ND -> (none)
- renumbered J5 to J7, U4 to U1
Connections:
- net +3.3V: now also J6.1 (Pin_1); no longer U1.1 (VBAT)
- net GND: now also B1.1, C5.2, R10.2; no longer U1.60 (BOOT0)
- new net: B1.2, U1.1 (VBAT)
- new net BOOT0: C5.1, J6.2 (Pin_2), R10.1, U1.60 (BOOT0)
- no-connect marks 22 -> 23

Commit message: PCB düzenleme.
Parts:
- C10, C12, C5, C8, C9: Digikey (none) -> 3372-0805B104K500BDTR-ND
- C11, C13, C6, C7: Digikey (none) -> 0805N100J101AD
- C14: Digikey (none) -> 0805B103K251DC
Changed lines of the file:
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@@
       (effects (font (size 1.27 1.27)) hide)
     )
-    (property "Digikey" "" (at 110.49 120.65 0)
+    (property "Digikey" "0805N100J101AD" (at 110.49 120.65 0)
       (effects (font (size 1.27 1.27)) hide)
     )
@@
       (effects (font (size 1.27 1.27)) hide)
     )
-    (property "Digikey" "" (at 120.65 120.65 0)
+    (property "Digikey" "0805N100J101AD" (at 120.65 120.65 0)
       (effects (font (size 1.27 1.27)) hide)
     )
@@
       (effects (font (size 1.27 1.27)) hide)
     )
-    (property "Digikey" "" (at 115.57 20.32 0)
+    (property "Digikey" "3372-0805B104K500BDTR-ND" (at 115.57 20.32 0)
       (effects (font (size 1.27 1.27)) hide)
     )
@@
       (effects (font (size 1.27 1.27)) hide)
     )
-    (property "Digikey" "" (at 64.77 80.01 0)
+    (property "Digikey" "0805N100J101AD" (at 64.77 80.01 0)
       (effects (font (size 1.27 1.27)) hide)
     )
@@
       (effects (font (size 1.27 1.27)) hide)
     )
-    (property "Digikey" "" (at 93.98 20.32 0)
+    (property "Digikey" "3372-0805B104K500BDTR-ND" (at 93.98 20.32 0)
       (effects (font (size 1.27 1.27)) hide)
     )
@@
       (effects (font (size 1.27 1.27)) hide)
     )
-    (property "Digikey" "" (at 54.61 80.01 0)
+    (property "Digikey" "0805N100J101AD" (at 54.61 80.01 0)
       (effects (font (size 1.27 1.27)) hide)
     )
@@
       (effects (font (size 1.27 1.27)) hide)
     )
-    (property "Digikey" "" (at 83.82 20.32 0)
+    (property "Digikey" "3372-0805B104K500BDTR-ND" (at 83.82 20.32 0)
       (effects (font (size 1.27 1.27)) hide)
     )
@@
       (effects (font (size 1.27 1.27)) hide)
     )
-    (property "Digikey" "" (at 31.75 43.18 0)
+    (property "Digikey" "3372-0805B104K500BDTR-ND" (at 31.75 43.18 0)
       (effects (font (size 1.27 1.27)) hide)
     )
@@
       (effects (font (size 1.27 1.27)) hide)
     )
-    (property "Digikey" "" (at 105.41 20.32 0)
+    (property "Digikey" "3372-0805B104K500BDTR-ND" (at 105.41 20.32 0)
       (effects (font (size 1.27 1.27)) hide)
     )
@@
       (effects (font (size 1.27 1.27)) hide)
     )
-    (property "Digikey" "" (at 125.73 20.32 0)
-      (effects (font (size 1.27 1.27)) hide)
-    )
+    (property "Digikey" "0805B103K251DC" (at 125.73 20.32 0)
+      (effects (font (size 1.27 1.27)) hide)
+    )
