File: hardware/rs232-rs485.kicad_sch (KiCad schematic)
At the start: 5 parts, among them U3 Max3075EESA

Commit message: Kicad şema düzenlemesi yapıldı.
Parts:
- added J?: Conn_02x01, Connector_Phoenix_MC:PhoenixContact_MCV_1,5_2-G-3.81_1x02_P3.81mm_Vertical, symbol Connector_Generic:Conn_02x01
- C20: renamed from C24; footprint Capacitor_SMD:C_0603_1608Metric -> Capacitor_SMD:C_0805_2012Metric
- renumbered R11 to R14, R17 to R15, R18 to R16
Connections:
- net RS485_A: no longer names the net of R15.2, U3.6 (A)
- net RS485_A: now also J?.1 (Pin_1)
- net RS485_B: no longer names the net of R16.1, U3.7 (B)
- net RS485_B: now also J?.2 (Pin_2)
- net RS485_EN renamed +5V

Commit message: PCB düzenleme.
Parts:
- C20: Digikey 311-1343-6-ND -> 3372-0805B104K500BDTR-ND
Changed lines of the file:
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@@
       (effects (font (size 1.27 1.27)) hide)
     )
-    (property "Digikey" "311-1343-6-ND" (at 167.64 82.55 0)
+    (property "Digikey" "3372-0805B104K500BDTR-ND" (at 167.64 82.55 0)
       (effects (font (size 1.27 1.27)) hide)
     )
