File: hardware/rs232.kicad_sch (KiCad schematic)
At the start: 0 parts

Commit message: Kicad şema düzenlemesi yapıldı.
Parts:
- added U5: MAX232N, N16, symbol drip-irrigation-sys-cc:MAX232N
Changed lines of the file:
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@@
 (kicad_sch (version 20230121) (generator eeschema)
   (paper "A4")
+  (symbol (lib_id "drip-irrigation-sys-cc:MAX232N") (at 127 78.74 0) (unit 1)
+    (in_bom yes) (on_board yes) (dnp no) (fields_autoplaced)
+    (property "Reference" "U5" (at 160.02 68.58 0)
+      (effects (font (size 1.524 1.524)))
+    )
+    (property "Value" "MAX232N" (at 160.02 71.12 0)
+      (effects (font (size 1.524 1.524)))
+    )
+    (property "Footprint" "N16" (at 127 78.74 0)
+      (effects (font (size 1.27 1.27) italic) hide)
+    )
+    (property "Datasheet" "MAX232N" (at 163.83 74.93 0)
+      (effects (font (size 1.27 1.27) italic) hide)
+    )
+    (property "Digikey" "296-1402-5-ND" (at 127 78.74 0)
+      (effects (font (size 1.27 1.27)) hide)
+    )
+    (pin "1")
+    (pin "10")
+    (pin "11")
+    (pin "12")
+    (pin "13")
+    (pin "14")
+    (pin "15")
+    (pin "16")
+    (pin "2")
+    (pin "3")
+    (pin "4")
+    (pin "5")
+    (pin "6")
+    (pin "7")
+    (pin "8")
+    (pin "9")
+    (instances
+      (project "drip-irrigation-sys-cc"
+        (path "/41708c1e-19b2-4374-83f2-108076d82b45/3f2f58a7-db97-4667-aa97-3e4409f949c8"
+          (reference "U5") (unit 1)
+        )
+      )
+    )
+  )
 )

Commit message: Kicad şema düzenlemesi yapıldı.
Parts:
- removed U5: MAX232N, N16, symbol drip-irrigation-sys-cc:MAX232N
- added C25, C26, C27, C28, C29: 100nF, Capacitor_SMD:C_0603_1608Metric, symbol Device:C
- added U6: MAX3222EWN_T, MAX3222EWN_T:SOIC127P1032X265-18N, symbol drip-irrigation-sys-cc:MAX3222EWN_T
Connections:
- new net: C28.1, U6.3 (V+)
- new net: C27.1, U6.7 (V-)
- new net: C26.1, U6.2 (C1+)
- new net: C26.2, U6.4 (C1-)
- new net: C25.1, U6.5 (C2+)
- new net: C25.2, U6.6 (C2-)
- new net +3V3: C29.1, U6.17 (VCC), U6.18 (~{SHDN})
- new net GND: C27.2, C28.2, C29.2, U6.1 (~{EN}), U6.16 (GND)
- new net RS232_RX: U6.14 (R1IN)
- new net RS232_TX: U6.15 (T1OUT)
- new net USART1_RX: U6.13 (R1OUT)
- new net USART1_TX: U6.12 (T1IN)
- no-connect marks 0 -> 4

Commit message: Kicad şema düzenlemesi yapıldı.
Parts:
- U6: Digikey (none) -> MAX3222EWN+TTR-ND
Changed lines of the file:
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@@
     (stroke (width 0) (type default))
-  )
-  (global_label "USART1_TX" (shape input) (at 191.77 64.77 180)
-    (effects (font (size 1.27 1.27)) (justify right))
-    (property "Intersheetrefs" "${INTERSHEET_REFS}" (at 191.77 64.77 0)
-      (effects (font (size 1.27 1.27)) hide)
-    )
-  )
-  (global_label "USART1_RX" (shape input) (at 229.87 57.15 0)
-    (effects (font (size 1.27 1.27)) (justify left))
-    (property "Intersheetrefs" "${INTERSHEET_REFS}" (at 229.87 57.15 0)
-      (effects (font (size 1.27 1.27)) hide)
-    )
   )
   (hierarchical_label "RS232_TX" (shape output) (at 229.87 64.77 0) (fields_autoplaced)
     (effects (font (size 1.27 1.27)) (justify left))
   )
+  (hierarchical_label "USART1_TX" (shape input) (at 191.77 64.77 180) (fields_autoplaced)
+    (effects (font (size 1.27 1.27)) (justify right))
+  )
   (hierarchical_label "RS232_RX" (shape input) (at 191.77 57.15 180) (fields_autoplaced)
     (effects (font (size 1.27 1.27)) (justify right))
+  )
+  (hierarchical_label "USART1_RX" (shape input) (at 229.87 57.15 0) (fields_autoplaced)
+    (effects (font (size 1.27 1.27)) (justify left))
   )
   (symbol (lib_id "Device:C") (at 250.19 54.61 0) (unit 1)
@@
       (effects (font (size 1.27 1.27)) (justify bottom) hide)
     )
-    (pin "1")
+    (property "Digikey" "MAX3222EWN+TTR-ND" (at 210.82 67.31 0)
+      (effects (font (size 1.27 1.27)) hide)
+    )
+    (pin "1")

Commit message: Kicad şema düzenlemesi yapıldı.
Parts:
- C?: renamed from C28; footprint Capacitor_SMD:C_0603_1608Metric -> Capacitor_SMD:C_0805_2012Metric
- C?: renamed from C27; footprint Capacitor_SMD:C_0603_1608Metric -> Capacitor_SMD:C_0805_2012Metric
- C?: renamed from C29; footprint Capacitor_SMD:C_0603_1608Metric -> Capacitor_SMD:C_0805_2012Metric
- C?: renamed from C26; footprint Capacitor_SMD:C_0603_1608Metric -> Capacitor_SMD:C_0805_2012Metric
- C?: renamed from C25; footprint Capacitor_SMD:C_0603_1608Metric -> Capacitor_SMD:C_0805_2012Metric
- renumbered U6 to U?

Commit message: PCB düzenlemesi yapıldı.
Parts:
- U?: footprint MAX3222EWN_T:SOIC127P1032X265-18N -> drip-irrigation-sys-cc:MAX3222EWN+T
Changed lines of the file:
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@@
       (effects (font (size 1.27 1.27)))
     )
-    (property "Footprint" "MAX3222EWN_T:SOIC127P1032X265-18N" (at 210.82 67.31 0)
+    (property "Footprint" "drip-irrigation-sys-cc:MAX3222EWN+T" (at 210.82 67.31 0)
       (effects (font (size 1.27 1.27)) (justify bottom) hide)
     )

Commit message: PCB düzenleme.
Parts:
- C? (x5): Digikey 311-1343-6-ND -> 3372-0805B104K500BDTR-ND
Changed lines of the file:
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@@
       (effects (font (size 1.27 1.27)) hide)
     )
-    (property "Digikey" "311-1343-6-ND" (at 250.19 54.61 0)
+    (property "Digikey" "3372-0805B104K500BDTR-ND" (at 250.19 54.61 0)
       (effects (font (size 1.27 1.27)) hide)
     )
@@
       (effects (font (size 1.27 1.27)) hide)
     )
-    (property "Digikey" "311-1343-6-ND" (at 242.57 80.01 0)
+    (property "Digikey" "3372-0805B104K500BDTR-ND" (at 242.57 80.01 0)
       (effects (font (size 1.27 1.27)) hide)
     )
@@
       (effects (font (size 1.27 1.27)) hide)
     )
-    (property "Digikey" "311-1343-6-ND" (at 260.35 54.61 0)
+    (property "Digikey" "3372-0805B104K500BDTR-ND" (at 260.35 54.61 0)
       (effects (font (size 1.27 1.27)) hide)
     )
@@
       (effects (font (size 1.27 1.27)) hide)
     )
-    (property "Digikey" "311-1343-6-ND" (at 186.69 73.66 0)
+    (property "Digikey" "3372-0805B104K500BDTR-ND" (at 186.69 73.66 0)
       (effects (font (size 1.27 1.27)) hide)
     )
@@
       (effects (font (size 1.27 1.27)) hide)
     )
-    (property "Digikey" "311-1343-6-ND" (at 173.99 81.28 0)
-      (effects (font (size 1.27 1.27)) hide)
-    )
+    (property "Digikey" "3372-0805B104K500BDTR-ND" (at 173.99 81.28 0)
+      (effects (font (size 1.27 1.27)) hide)
+    )
